Commit message: Update base_link visual configs

File: src/motion/manipulator/urdf/arcsys2.urdf (robot description, URDF)
Before this commit: robot arcsys2, 2 links, 1 joints
Links:
- link base_link: geometry visual box size=0.3 0.3 1.0

Commit message: Change base_link visual size

File: src/motion/manipulator/urdf/arcsys2.urdf (robot description, URDF)
Before this commit: robot arcsys2, 2 links, 1 joints
Links:
- link base_link: geometry visual box size=1.0 1.0 1.0

Commit message: Change joint name

File: src/motion/manipulator/urdf/arcsys2.urdf (robot description, URDF)
Before this commit: robot arcsys2, 2 links, 1 joints
Joints:
- removed joint fixed_base2shaft
- added joint base2shaft: type fixed, parent base_link, child main_shaft

Commit message: Change size of main_shaft

File: src/motion/manipulator/urdf/arcsys2.urdf (robot description, URDF)
Before this commit: robot arcsys2, 2 links, 1 joints
Links:
- link main_shaft: geometry visual box size=0.3 0.3 1.0
