Commit message: Clean up files

File: src/motion/manipulator/urdf/arcsys2.xacro (robot description, xacro)
@@ -6,17 +6,19 @@
   <material name="blue">  <color rgba="${  0/255} ${  0/255} ${255/255} 1.0"/> </material>
   <xacro:LINK name="world">
-    <origin xyz="0.0 0.0 0.0" rpy="0.0 0.0 0.0"/>
+    <origin xyz="0 0 0" rpy="0 0 0"/>
   </xacro:LINK>
   <xacro:FIXED_JOINT parent="world" child="rail"/>
-  <xacro:LINK name="rail" width="10.0" depth="0.3" height="0.1" color="blue">
-    <origin xyz="0.0 0.0 0.05" rpy="0.0 0.0 0.0"/>
+  <xacro:property name="rail_height" value="0.1"/>
+  <xacro:LINK name="rail" width="10.0" depth="0.3" height="${rail_height}" color="blue">
+    <origin xyz="0 0 ${rail_height/2}" rpy="0 0 0"/>
   </xacro:LINK>
   <xacro:PRISMATIC_JOINT parent="rail" child="base" x="1" lower="-5.0" upper="5.0"/>
-  <xacro:LINK name="base" width="0.3" depth="0.3" height="1.0" color="red">
-    <origin xyz="0.0 0.0 0.75" rpy="0.0 0.0 0.0"/>
+  <xacro:property name="base_height" value="2.0"/>
+  <xacro:LINK name="base" width="0.1" depth="0.1" height="${base_height}" color="red">
+    <origin xyz="0 0 ${base_height/2}" rpy="0 0 0"/>
   </xacro:LINK>
   <xacro:PRISMATIC_JOINT parent="base" child="arm0" z="1" lower="-0.5" upper="0.5"/>
   <xacro:LINK name="arm0" width="0.2" depth="0.5" height="0.2" color="red">
-    <origin xyz="0.0 0.15 1.5" rpy="0.0 0.0 0.0"/>
+    <origin xyz="0 0.15 1.5" rpy="0 0 0"/>
   </xacro:LINK>
   <xacro:macro name="LINK" params="name *origin width:=0.0 depth:=0.0 height:=0.0 color:=white">
@@ -40,4 +42,5 @@
   <xacro:macro name="PRISMATIC_JOINT" params="parent child x:=0 y:=0 z:=0 lower upper">
     <joint name="${parent}->${child}" type="prismatic">
+      <origin xyz="0 0 0" rpy="0 0 0"/>
       <parent link="${parent}"/>
       <child link="${child}"/>

Commit message: Change some literals to xacro:property

File: src/motion/manipulator/urdf/arcsys2.xacro (robot description, xacro)
@@ -14,11 +14,15 @@
   </xacro:LINK>
   <xacro:PRISMATIC_JOINT parent="rail" child="base" x="1" lower="-5.0" upper="5.0"/>
+  <xacro:property name="base_thickness" value="0.1"/>
   <xacro:property name="base_height" value="2.0"/>
-  <xacro:LINK name="base" width="0.1" depth="0.1" height="${base_height}" color="red">
+  <xacro:LINK name="base" width="${base_thickness}" depth="${base_thickness}" height="${base_height}" color="red">
     <origin xyz="0 0 ${base_height/2}" rpy="0 0 0"/>
   </xacro:LINK>
   <xacro:PRISMATIC_JOINT parent="base" child="arm0" z="1" lower="-0.5" upper="0.5"/>
-  <xacro:LINK name="arm0" width="0.2" depth="0.5" height="0.2" color="red">
-    <origin xyz="0 0.15 1.5" rpy="0 0 0"/>
+  <xacro:property name="arm_width" value="0.1"/>
+  <xacro:property name="arm_depth" value="0.5"/>
+  <xacro:property name="arm_height" value="${arm_width}"/>
+  <xacro:LINK name="arm0" width="${arm_width}" depth="${arm_depth}" height="${arm_height}" color="red">
+    <origin xyz="0 ${base_thickness} ${base_height*0.75}" rpy="0 0 0"/>
   </xacro:LINK>
   <xacro:macro name="LINK" params="name *origin width:=0.0 depth:=0.0 height:=0.0 color:=white">

Commit message: Change link name "base" to "shaft"

File: src/motion/manipulator/urdf/arcsys2.xacro (robot description, xacro)
@@ -13,16 +13,16 @@
     <origin xyz="0 0 ${rail_height/2}" rpy="0 0 0"/>
   </xacro:LINK>
-  <xacro:PRISMATIC_JOINT parent="rail" child="base" x="1" lower="-5.0" upper="5.0"/>
-  <xacro:property name="base_thickness" value="0.1"/>
-  <xacro:property name="base_height" value="2.0"/>
-  <xacro:LINK name="base" width="${base_thickness}" depth="${base_thickness}" height="${base_height}" color="red">
-    <origin xyz="0 0 ${base_height/2}" rpy="0 0 0"/>
+  <xacro:PRISMATIC_JOINT parent="rail" child="shaft" x="1" lower="-5.0" upper="5.0"/>
+  <xacro:property name="shaft_thickness" value="0.1"/>
+  <xacro:property name="shaft_height" value="2.0"/>
+  <xacro:LINK name="shaft" width="${shaft_thickness}" depth="${shaft_thickness}" height="${shaft_height}" color="red">
+    <origin xyz="0 0 ${shaft_height/2}" rpy="0 0 0"/>
   </xacro:LINK>
-  <xacro:PRISMATIC_JOINT parent="base" child="arm0" z="1" lower="-0.5" upper="0.5"/>
+  <xacro:PRISMATIC_JOINT parent="shaft" child="arm0" z="1" lower="-0.5" upper="0.5"/>
   <xacro:property name="arm_width" value="0.1"/>
   <xacro:property name="arm_depth" value="0.5"/>
   <xacro:property name="arm_height" value="${arm_width}"/>
   <xacro:LINK name="arm0" width="${arm_width}" depth="${arm_depth}" height="${arm_height}" color="red">
-    <origin xyz="0 ${base_thickness} ${base_height*0.75}" rpy="0 0 0"/>
+    <origin xyz="0 ${shaft_thickness} ${shaft_height*0.75}" rpy="0 0 0"/>
   </xacro:LINK>
   <xacro:macro name="LINK" params="name *origin width:=0.0 depth:=0.0 height:=0.0 color:=white">

Commit message: Delete link "rail"

File: src/motion/manipulator/urdf/arcsys2.xacro (robot description, xacro)
@@ -8,10 +8,5 @@
     <origin xyz="0 0 0" rpy="0 0 0"/>
   </xacro:LINK>
-  <xacro:FIXED_JOINT parent="world" child="rail"/>
-  <xacro:property name="rail_height" value="0.1"/>
-  <xacro:LINK name="rail" width="10.0" depth="0.3" height="${rail_height}" color="blue">
-    <origin xyz="0 0 ${rail_height/2}" rpy="0 0 0"/>
-  </xacro:LINK>
-  <xacro:PRISMATIC_JOINT parent="rail" child="shaft" x="1" lower="-5.0" upper="5.0"/>
+  <xacro:PRISMATIC_JOINT parent="world" child="shaft" x="1" lower="-5.0" upper="5.0"/>
   <xacro:property name="shaft_thickness" value="0.1"/>
   <xacro:property name="shaft_height" value="2.0"/>

Commit message: Change PRISMATIC_JOINT to LIMITED_JOINT
prismaticなジョイントを作った後にrevoluteなジョイントを作ろうとしたら
どちらもlimited要素を持つ全くtype以外全く同じ要素のジョイントだったため，
prismaticを改名

File: src/motion/manipulator/urdf/arcsys2.xacro (robot description, xacro)
@@ -8,16 +8,21 @@
     <origin xyz="0 0 0" rpy="0 0 0"/>
   </xacro:LINK>
-  <xacro:PRISMATIC_JOINT parent="world" child="shaft" x="1" lower="-5.0" upper="5.0"/>
+  <xacro:LIMITED_JOINT parent="world" child="shaft" type="prismatic" x="1" lower="-5.0" upper="5.0"/>
   <xacro:property name="shaft_thickness" value="0.1"/>
   <xacro:property name="shaft_height" value="2.0"/>
-  <xacro:LINK name="shaft" width="${shaft_thickness}" depth="${shaft_thickness}" height="${shaft_height}" color="red">
+  <xacro:LINK name="shaft" width="${shaft_thickness}" depth="${shaft_thickness}" height="${shaft_height}" color="black">
     <origin xyz="0 0 ${shaft_height/2}" rpy="0 0 0"/>
   </xacro:LINK>
-  <xacro:PRISMATIC_JOINT parent="shaft" child="arm0" z="1" lower="-0.5" upper="0.5"/>
+  <xacro:LIMITED_JOINT parent="shaft" child="arm0" type="prismatic" z="1" lower="-0.5" upper="0.5"/>
   <xacro:property name="arm_width" value="0.1"/>
   <xacro:property name="arm_depth" value="0.5"/>
   <xacro:property name="arm_height" value="${arm_width}"/>
-  <xacro:LINK name="arm0" width="${arm_width}" depth="${arm_depth}" height="${arm_height}" color="red">
+  <xacro:LINK name="arm0" width="${arm_width}" depth="${arm_depth}" height="${arm_height}">
     <origin xyz="0 ${shaft_thickness} ${shaft_height*0.75}" rpy="0 0 0"/>
+  </xacro:LINK>
+  <xacro:property name="pi" value="3.1415"/>
+  <xacro:LIMITED_JOINT parent="arm0" child="arm1" type="revolute" z="1" lower="${-pi}" upper="${pi}"/>
+  <xacro:LINK name="arm1" width="${arm_width}" depth="${arm_depth}" height="${arm_height}" color="black">
+    <origin xyz="0 ${shaft_thickness+arm_depth} ${shaft_height*0.75}" rpy="0 0 0"/>
   </xacro:LINK>
   <xacro:macro name="LINK" params="name *origin width:=0.0 depth:=0.0 height:=0.0 color:=white">
@@ -32,5 +37,5 @@
     </link>
   </xacro:macro>
-  <xacro:macro name="FIXED_JOINT" params="parent child">
+  <!--xacro:macro name="FIXED_JOINT" params="parent child">
     <joint name="${parent}->${child}" type="fixed">
       <origin xyz="0 0 0" rpy="0 0 0"/>
@@ -38,8 +43,8 @@
       <child link="${child}"/>
     </joint>
-  </xacro:macro>
-  <xacro:macro name="PRISMATIC_JOINT" params="parent child x:=0 y:=0 z:=0 lower upper">
-    <joint name="${parent}->${child}" type="prismatic">
-      <origin xyz="0 0 0" rpy="0 0 0"/>
+  </xacro:macro-->
+  <xacro:macro name="LIMITED_JOINT" params="parent child type x:=0 y:=0 z:=0 lower upper *origin">
+    <joint name="${parent}->${child}" type="${type}">
+      <xacro:insert_block name="origin"/>
       <parent link="${parent}"/>
       <child link="${child}"/>

Commit message: Save point
内容は途中保存

File: src/motion/manipulator/urdf/arcsys2.xacro (robot description, xacro)
@@ -8,5 +8,7 @@
     <origin xyz="0 0 0" rpy="0 0 0"/>
   </xacro:LINK>
-  <xacro:LIMITED_JOINT parent="world" child="shaft" type="prismatic" x="1" lower="-5.0" upper="5.0"/>
+  <xacro:LIMITED_JOINT parent="world" child="shaft" type="prismatic" x="1" lower="-5.0" upper="5.0">
+    <origin xyz="0 0 0" rpy="0 0 0"/>
+  </xacro:LIMITED_JOINT>
   <xacro:property name="shaft_thickness" value="0.1"/>
   <xacro:property name="shaft_height" value="2.0"/>
@@ -14,17 +16,21 @@
     <origin xyz="0 0 ${shaft_height/2}" rpy="0 0 0"/>
   </xacro:LINK>
-  <xacro:LIMITED_JOINT parent="shaft" child="arm0" type="prismatic" z="1" lower="-0.5" upper="0.5"/>
+  <xacro:LIMITED_JOINT parent="shaft" child="arm0" type="prismatic" z="1" lower="-0.5" upper="0.5">
+    <origin xyz="0 0 0" rpy="0 0 0"/>
+  </xacro:LIMITED_JOINT>
   <xacro:property name="arm_width" value="0.1"/>
   <xacro:property name="arm_depth" value="0.5"/>
   <xacro:property name="arm_height" value="${arm_width}"/>
   <xacro:LINK name="arm0" width="${arm_width}" depth="${arm_depth}" height="${arm_height}">
-    <origin xyz="0 ${shaft_thickness} ${shaft_height*0.75}" rpy="0 0 0"/>
+    <origin xyz="0 ${shaft_thickness/2 + arm_depth/2} ${shaft_height*0.75}" rpy="0 0 0"/>
   </xacro:LINK>
   <xacro:property name="pi" value="3.1415"/>
-  <xacro:LIMITED_JOINT parent="arm0" child="arm1" type="revolute" z="1" lower="${-pi}" upper="${pi}"/>
+  <xacro:LIMITED_JOINT parent="arm0" child="arm1" type="revolute" z="1">
+    <origin xyz="0 ${shaft_thickness/2 + arm_depth} 0" rpy="0 0 0"/>
+  </xacro:LIMITED_JOINT>
   <xacro:LINK name="arm1" width="${arm_width}" depth="${arm_depth}" height="${arm_height}" color="black">
-    <origin xyz="0 ${shaft_thickness+arm_depth} ${shaft_height*0.75}" rpy="0 0 0"/>
+    <origin xyz="0 ${shaft_thickness/2 + arm_depth*0.75} ${shaft_height*0.75}" rpy="0 0 0"/>
   </xacro:LINK>
-  <xacro:macro name="LINK" params="name *origin width:=0.0 depth:=0.0 height:=0.0 color:=white">
+  <xacro:macro name="LINK" params="name *origin width:=0 depth:=0 height:=0 color:=white">
     <link name="${name}">
       <visual>
@@ -37,12 +43,5 @@
     </link>
   </xacro:macro>
-  <!--xacro:macro name="FIXED_JOINT" params="parent child">
-    <joint name="${parent}->${child}" type="fixed">
-      <origin xyz="0 0 0" rpy="0 0 0"/>
-      <parent link="${parent}"/>
-      <child link="${child}"/>
-    </joint>
-  </xacro:macro-->
-  <xacro:macro name="LIMITED_JOINT" params="parent child type x:=0 y:=0 z:=0 lower upper *origin">
+  <xacro:macro name="LIMITED_JOINT" params="parent child type x:=0 y:=0 z:=0 lower:=${-pi} upper:=${pi} *origin">
     <joint name="${parent}->${child}" type="${type}">
       <xacro:insert_block name="origin"/>
@@ -50,5 +49,5 @@
       <child link="${child}"/>
       <axis xyz="${x} ${y} ${z}"/>
-      <limit lower="${lower}" upper="${upper}" effort="1.0" velocity="1.0"/>
+      <limit lower="${lower}" upper="${upper}" effort="1" velocity="1"/>
     </joint>
   </xacro:macro>

Commit message: Change xacro:macro name

File: src/motion/manipulator/urdf/arcsys2.xacro (robot description, xacro)
@@ -8,7 +8,7 @@
     <origin xyz="0 0 0" rpy="0 0 0"/>
   </xacro:LINK>
-  <xacro:LIMITED_JOINT parent="world" child="shaft" type="prismatic" x="1" lower="-5.0" upper="5.0">
+  <xacro:JOINT parent="world" child="shaft" type="prismatic" x="1" lower="-5.0" upper="5.0">
     <origin xyz="0 0 0" rpy="0 0 0"/>
-  </xacro:LIMITED_JOINT>
+  </xacro:JOINT>
   <xacro:property name="shaft_thickness" value="0.1"/>
   <xacro:property name="shaft_height" value="2.0"/>
@@ -16,7 +16,7 @@
     <origin xyz="0 0 ${shaft_height/2}" rpy="0 0 0"/>
   </xacro:LINK>
-  <xacro:LIMITED_JOINT parent="shaft" child="arm0" type="prismatic" z="1" lower="-0.5" upper="0.5">
+  <xacro:JOINT parent="shaft" child="arm0" type="prismatic" z="1" lower="-0.5" upper="0.5">
     <origin xyz="0 0 0" rpy="0 0 0"/>
-  </xacro:LIMITED_JOINT>
+  </xacro:JOINT>
   <xacro:property name="arm_width" value="0.1"/>
   <xacro:property name="arm_depth" value="0.5"/>
@@ -26,7 +26,7 @@
   </xacro:LINK>
   <xacro:property name="pi" value="3.1415"/>
-  <xacro:LIMITED_JOINT parent="arm0" child="arm1" type="revolute" z="1">
+  <xacro:JOINT parent="arm0" child="arm1" type="revolute" z="1">
     <origin xyz="0 ${shaft_thickness/2 + arm_depth} 0" rpy="0 0 0"/>
-  </xacro:LIMITED_JOINT>
+  </xacro:JOINT>
   <xacro:LINK name="arm1" width="${arm_width}" depth="${arm_depth}" height="${arm_height}" color="black">
     <origin xyz="0 ${shaft_thickness/2 + arm_depth*0.75} ${shaft_height*0.75}" rpy="0 0 0"/>
@@ -43,5 +43,5 @@
     </link>
   </xacro:macro>
-  <xacro:macro name="LIMITED_JOINT" params="parent child type x:=0 y:=0 z:=0 lower:=${-pi} upper:=${pi} *origin">
+  <xacro:macro name="JOINT" params="parent child type x:=0 y:=0 z:=0 lower:=${-pi} upper:=${pi} *origin">
     <joint name="${parent}->${child}" type="${type}">
       <xacro:insert_block name="origin"/>

Commit message: Change coordinate system

File: src/motion/manipulator/urdf/arcsys2.xacro (robot description, xacro)
@@ -1,41 +1,49 @@
 <?xml version="1.0"?>
 <robot xmlns:xacro="http://ros.org/wiki/xacro" name="arcsys2">
-  <material name="white"> <color rgba="${255/255} ${255/255} ${255/255} 1.0"/> </material>
-  <material name="red">   <color rgba="${255/255} ${  0/255} ${  0/255} 1.0"/> </material>
-  <material name="green"> <color rgba="${  0/255} ${255/255} ${  0/255} 1.0"/> </material>
-  <material name="blue">  <color rgba="${  0/255} ${  0/255} ${255/255} 1.0"/> </material>
+  <material name="white"> <color rgba="${255/255} ${255/255} ${255/255} 1.0" /> </material>
+  <material name="red">   <color rgba="${255/255} ${  0/255} ${  0/255} 1.0" /> </material>
+  <material name="green"> <color rgba="${  0/255} ${255/255} ${  0/255} 1.0" /> </material>
+  <material name="blue">  <color rgba="${  0/255} ${  0/255} ${255/255} 1.0" /> </material>
   <xacro:LINK name="world">
-    <origin xyz="0 0 0" rpy="0 0 0"/>
+    <origin xyz="0 0 0" />
   </xacro:LINK>
-  <xacro:JOINT parent="world" child="shaft" type="prismatic" x="1" lower="-5.0" upper="5.0">
-    <origin xyz="0 0 0" rpy="0 0 0"/>
+  <xacro:property name="shaft_height" value="2.0"/>
+  <xacro:JOINT parent="world" child="shaft" type="prismatic" y="1" lower="-5.0" upper="5.0">
+    <origin xyz="0 0 ${shaft_height/2}" rpy="0 0 0" />
   </xacro:JOINT>
   <xacro:property name="shaft_thickness" value="0.1"/>
-  <xacro:property name="shaft_height" value="2.0"/>
-  <xacro:LINK name="shaft" width="${shaft_thickness}" depth="${shaft_thickness}" height="${shaft_height}" color="black">
-    <origin xyz="0 0 ${shaft_height/2}" rpy="0 0 0"/>
+  <xacro:LINK name="shaft" width="${shaft_thickness}" depth="${shaft_thickness}" height="${shaft_height}" color="red">
+    <origin xyz="0 0 0" />
   </xacro:LINK>
+  <xacro:property name="arm0_depth" value="0.1"/>
   <xacro:JOINT parent="shaft" child="arm0" type="prismatic" z="1" lower="-0.5" upper="0.5">
-    <origin xyz="0 0 0" rpy="0 0 0"/>
+    <origin xyz="${shaft_thickness/2 + arm0_depth/2} 0 ${shaft_height/4}" rpy="0 0 0"/>
   </xacro:JOINT>
   <xacro:property name="arm_width" value="0.1"/>
-  <xacro:property name="arm_depth" value="0.5"/>
   <xacro:property name="arm_height" value="${arm_width}"/>
-  <xacro:LINK name="arm0" width="${arm_width}" depth="${arm_depth}" height="${arm_height}">
-    <origin xyz="0 ${shaft_thickness/2 + arm_depth/2} ${shaft_height*0.75}" rpy="0 0 0"/>
+  <xacro:LINK name="arm0" width="${arm_width}" depth="${arm0_depth}" height="${arm_height}" color="green">
+    <origin xyz="0 0 0"/>
   </xacro:LINK>
   <xacro:property name="pi" value="3.1415"/>
   <xacro:JOINT parent="arm0" child="arm1" type="revolute" z="1">
-    <origin xyz="0 ${shaft_thickness/2 + arm_depth} 0" rpy="0 0 0"/>
+    <origin xyz="${arm0_depth/2} 0 0" rpy="0 0 0"/>
   </xacro:JOINT>
-  <xacro:LINK name="arm1" width="${arm_width}" depth="${arm_depth}" height="${arm_height}" color="black">
-    <origin xyz="0 ${shaft_thickness/2 + arm_depth*0.75} ${shaft_height*0.75}" rpy="0 0 0"/>
+  <xacro:property name="arm1_depth" value="0.5"/>
+  <xacro:LINK name="arm1" width="${arm_width}" depth="${arm1_depth}" height="${arm_height}" color="blue">
+    <origin xyz="${arm1_depth/2} 0 0" />
   </xacro:LINK>
-  <xacro:macro name="LINK" params="name *origin width:=0 depth:=0 height:=0 color:=white">
+  <xacro:JOINT parent="arm1" child="arm2" type="revolute" z="1">
+    <origin xyz="${arm1_depth} 0 0" rpy="0 0 0"/>
+  </xacro:JOINT>
+  <xacro:property name="arm2_depth" value="0.5"/>
+  <xacro:LINK name="arm2" width="${arm_width}" depth="${arm2_depth}" height="${arm_height}" color="red">
+    <origin xyz="${arm2_depth/2} 0 0" />
+  </xacro:LINK>
+  <xacro:macro name="LINK" params="name width:=0 depth:=0 height:=0 color:=white *origin">
     <link name="${name}">
       <visual>
         <xacro:insert_block name="origin"/>
         <geometry>
-          <box size="${width} ${depth} ${height}"/>
+          <box size="${depth} ${width} ${height}"/>
         </geometry>
         <material name="${color}"/>
@@ -43,5 +51,5 @@
     </link>
   </xacro:macro>
-  <xacro:macro name="JOINT" params="parent child type x:=0 y:=0 z:=0 lower:=${-pi} upper:=${pi} *origin">
+  <xacro:macro name="JOINT" params="parent child type x:=0 y:=0 z:=0 lower:=${-pi/2} upper:=${pi/2} *origin">
     <joint name="${parent}->${child}" type="${type}">
       <xacro:insert_block name="origin"/>

Commit message: Devide property from LINK and JOINT definition

File: src/motion/manipulator/urdf/arcsys2.xacro (robot description, xacro)
@@ -5,29 +5,30 @@
   <material name="green"> <color rgba="${  0/255} ${255/255} ${  0/255} 1.0" /> </material>
   <material name="blue">  <color rgba="${  0/255} ${  0/255} ${255/255} 1.0" /> </material>
+  <xacro:property name="pi" value="3.1415"/>
+  <xacro:property name="shaft_height" value="2.0"/>
+  <xacro:property name="shaft_thickness" value="0.1"/>
+  <xacro:property name="arm_width" value="0.1"/>
+  <xacro:property name="arm_height" value="${arm_width}"/>
+  <xacro:property name="arm0_depth" value="0.1"/>
+  <xacro:property name="arm1_depth" value="0.5"/>
+  <xacro:property name="arm2_depth" value="0.5"/>
   <xacro:LINK name="world">
     <origin xyz="0 0 0" />
   </xacro:LINK>
-  <xacro:property name="shaft_height" value="2.0"/>
   <xacro:JOINT parent="world" child="shaft" type="prismatic" y="1" lower="-5.0" upper="5.0">
     <origin xyz="0 0 ${shaft_height/2}" rpy="0 0 0" />
   </xacro:JOINT>
-  <xacro:property name="shaft_thickness" value="0.1"/>
   <xacro:LINK name="shaft" width="${shaft_thickness}" depth="${shaft_thickness}" height="${shaft_height}" color="red">
     <origin xyz="0 0 0" />
   </xacro:LINK>
-  <xacro:property name="arm0_depth" value="0.1"/>
   <xacro:JOINT parent="shaft" child="arm0" type="prismatic" z="1" lower="-0.5" upper="0.5">
     <origin xyz="${shaft_thickness/2 + arm0_depth/2} 0 ${shaft_height/4}" rpy="0 0 0"/>
   </xacro:JOINT>
-  <xacro:property name="arm_width" value="0.1"/>
-  <xacro:property name="arm_height" value="${arm_width}"/>
   <xacro:LINK name="arm0" width="${arm_width}" depth="${arm0_depth}" height="${arm_height}" color="green">
     <origin xyz="0 0 0"/>
   </xacro:LINK>
-  <xacro:property name="pi" value="3.1415"/>
   <xacro:JOINT parent="arm0" child="arm1" type="revolute" z="1">
     <origin xyz="${arm0_depth/2} 0 0" rpy="0 0 0"/>
   </xacro:JOINT>
-  <xacro:property name="arm1_depth" value="0.5"/>
   <xacro:LINK name="arm1" width="${arm_width}" depth="${arm1_depth}" height="${arm_height}" color="blue">
     <origin xyz="${arm1_depth/2} 0 0" />
@@ -36,5 +37,4 @@
     <origin xyz="${arm1_depth} 0 0" rpy="0 0 0"/>
   </xacro:JOINT>
-  <xacro:property name="arm2_depth" value="0.5"/>
   <xacro:LINK name="arm2" width="${arm_width}" depth="${arm2_depth}" height="${arm_height}" color="red">
     <origin xyz="${arm2_depth/2} 0 0" />
