Commit message: Change world "depth" to "length"

File: src/motion/manipulator/urdf/arcsys2.xacro (robot description, xacro)
@@ -10,7 +10,7 @@
   <xacro:property name="arm_width" value="0.1"/>
   <xacro:property name="arm_height" value="${arm_width}"/>
-  <xacro:property name="arm0_depth" value="0.1"/>
-  <xacro:property name="arm1_depth" value="0.5"/>
-  <xacro:property name="arm2_depth" value="0.5"/>
+  <xacro:property name="arm0_length" value="0.1"/>
+  <xacro:property name="arm1_length" value="0.5"/>
+  <xacro:property name="arm2_length" value="0.5"/>
   <xacro:LINK name="world">
     <origin xyz="0 0 0" />
@@ -19,31 +19,31 @@
     <origin xyz="0 0 ${shaft_height/2}" rpy="0 0 0" />
   </xacro:JOINT>
-  <xacro:LINK name="shaft" width="${shaft_thickness}" depth="${shaft_thickness}" height="${shaft_height}" color="red">
+  <xacro:LINK name="shaft" width="${shaft_thickness}" length="${shaft_thickness}" height="${shaft_height}" color="red">
     <origin xyz="0 0 0" />
   </xacro:LINK>
   <xacro:JOINT parent="shaft" child="arm0" type="prismatic" z="1" lower="-0.5" upper="0.5">
-    <origin xyz="${shaft_thickness/2 + arm0_depth/2} 0 ${shaft_height/4}" rpy="0 0 0"/>
+    <origin xyz="${shaft_thickness/2 + arm0_length/2} 0 ${shaft_height/4}" rpy="0 0 0"/>
   </xacro:JOINT>
-  <xacro:LINK name="arm0" width="${arm_width}" depth="${arm0_depth}" height="${arm_height}" color="green">
+  <xacro:LINK name="arm0" width="${arm_width}" length="${arm0_length}" height="${arm_height}" color="green">
     <origin xyz="0 0 0"/>
   </xacro:LINK>
   <xacro:JOINT parent="arm0" child="arm1" type="revolute" z="1">
-    <origin xyz="${arm0_depth/2} 0 0" rpy="0 0 0"/>
+    <origin xyz="${arm0_length/2} 0 0" rpy="0 0 0"/>
   </xacro:JOINT>
-  <xacro:LINK name="arm1" width="${arm_width}" depth="${arm1_depth}" height="${arm_height}" color="blue">
-    <origin xyz="${arm1_depth/2} 0 0" />
+  <xacro:LINK name="arm1" width="${arm_width}" length="${arm1_length}" height="${arm_height}" color="blue">
+    <origin xyz="${arm1_length/2} 0 0" />
   </xacro:LINK>
   <xacro:JOINT parent="arm1" child="arm2" type="revolute" z="1">
-    <origin xyz="${arm1_depth} 0 0" rpy="0 0 0"/>
+    <origin xyz="${arm1_length} 0 0" rpy="0 0 0"/>
   </xacro:JOINT>
-  <xacro:LINK name="arm2" width="${arm_width}" depth="${arm2_depth}" height="${arm_height}" color="red">
-    <origin xyz="${arm2_depth/2} 0 0" />
+  <xacro:LINK name="arm2" width="${arm_width}" length="${arm2_length}" height="${arm_height}" color="red">
+    <origin xyz="${arm2_length/2} 0 0" />
   </xacro:LINK>
-  <xacro:macro name="LINK" params="name width:=0 depth:=0 height:=0 color:=white *origin">
+  <xacro:macro name="LINK" params="name width:=0 length:=0 height:=0 color:=white *origin">
     <link name="${name}">
       <visual>
         <xacro:insert_block name="origin"/>
         <geometry>
-          <box size="${depth} ${width} ${height}"/>
+          <box size="${length} ${width} ${height}"/>
         </geometry>
         <material name="${color}"/>

Commit message: Delete some unnecessary code

File: src/motion/manipulator/urdf/arcsys2.xacro (robot description, xacro)
@@ -17,11 +17,11 @@
   </xacro:LINK>
   <xacro:JOINT parent="world" child="shaft" type="prismatic" y="1" lower="-5.0" upper="5.0">
-    <origin xyz="0 0 ${shaft_height/2}" rpy="0 0 0" />
+    <origin xyz="0 0 ${shaft_height/2}"/>
   </xacro:JOINT>
   <xacro:LINK name="shaft" width="${shaft_thickness}" length="${shaft_thickness}" height="${shaft_height}" color="red">
-    <origin xyz="0 0 0" />
+    <origin xyz="0 0 0"/>
   </xacro:LINK>
   <xacro:JOINT parent="shaft" child="arm0" type="prismatic" z="1" lower="-0.5" upper="0.5">
-    <origin xyz="${shaft_thickness/2 + arm0_length/2} 0 ${shaft_height/4}" rpy="0 0 0"/>
+    <origin xyz="${shaft_thickness/2 + arm0_length/2} 0 ${shaft_height/4}"/>
   </xacro:JOINT>
   <xacro:LINK name="arm0" width="${arm_width}" length="${arm0_length}" height="${arm_height}" color="green">
@@ -29,14 +29,14 @@
   </xacro:LINK>
   <xacro:JOINT parent="arm0" child="arm1" type="revolute" z="1">
-    <origin xyz="${arm0_length/2} 0 0" rpy="0 0 0"/>
+    <origin xyz="${arm0_length/2} 0 0"/>
   </xacro:JOINT>
   <xacro:LINK name="arm1" width="${arm_width}" length="${arm1_length}" height="${arm_height}" color="blue">
-    <origin xyz="${arm1_length/2} 0 0" />
+    <origin xyz="${arm1_length/2} 0 0"/>
   </xacro:LINK>
   <xacro:JOINT parent="arm1" child="arm2" type="revolute" z="1">
-    <origin xyz="${arm1_length} 0 0" rpy="0 0 0"/>
+    <origin xyz="${arm1_length} 0 0"/>
   </xacro:JOINT>
   <xacro:LINK name="arm2" width="${arm_width}" length="${arm2_length}" height="${arm_height}" color="red">
-    <origin xyz="${arm2_length/2} 0 0" />
+    <origin xyz="${arm2_length/2} 0 0"/>
   </xacro:LINK>
   <xacro:macro name="LINK" params="name width:=0 length:=0 height:=0 color:=white *origin">

Commit message: Create new macro "SCARA_JOINT"

File: src/motion/manipulator/urdf/arcsys2.xacro (robot description, xacro)
@@ -23,18 +23,20 @@
   </xacro:LINK>
   <xacro:JOINT parent="shaft" child="arm0" type="prismatic" z="1" lower="-0.5" upper="0.5">
-    <origin xyz="${shaft_thickness/2 + arm0_length/2} 0 ${shaft_height/4}"/>
+    <origin xyz="${shaft_thickness/2} 0 ${shaft_height/4}"/>
   </xacro:JOINT>
   <xacro:LINK name="arm0" width="${arm_width}" length="${arm0_length}" height="${arm_height}" color="green">
-    <origin xyz="0 0 0"/>
+    <origin xyz="${arm0_length/2} 0 0"/>
   </xacro:LINK>
-  <xacro:JOINT parent="arm0" child="arm1" type="revolute" z="1">
-    <origin xyz="${arm0_length/2} 0 0"/>
-  </xacro:JOINT>
+  <!--xacro:JOINT parent="arm0" child="arm1" type="revolute" z="1">
+    <origin xyz="${arm0_length} 0 0"/>
+  </xacro:JOINT-->
+  <xacro:SCARA_JOINT parent="arm0" child="arm1" parent_length="${arm0_length}"/>
   <xacro:LINK name="arm1" width="${arm_width}" length="${arm1_length}" height="${arm_height}" color="blue">
     <origin xyz="${arm1_length/2} 0 0"/>
   </xacro:LINK>
-  <xacro:JOINT parent="arm1" child="arm2" type="revolute" z="1">
+  <!--xacro:JOINT parent="arm1" child="arm2" type="revolute" z="1">
     <origin xyz="${arm1_length} 0 0"/>
-  </xacro:JOINT>
+  </xacro:JOINT-->
+  <xacro:SCARA_JOINT parent="arm1" child="arm2" parent_length="${arm1_length}"/>
   <xacro:LINK name="arm2" width="${arm_width}" length="${arm2_length}" height="${arm_height}" color="red">
     <origin xyz="${arm2_length/2} 0 0"/>
@@ -60,3 +62,12 @@
     </joint>
   </xacro:macro>
+  <xacro:macro name="SCARA_JOINT" params="parent child parent_length lower:=${-pi/2} upper:=${pi/2}">
+    <joint name="${parent}->${child}" type="revolute">
+      <origin xyz="${parent_length} 0 0"/>
+      <parent link="${parent}"/>
+      <child link="${child}"/>
+      <axis xyz="0 0 1"/>
+      <limit lower="${lower}" upper="${upper}" effort="1" velocity="1"/>
+    </joint>
+  </xacro:macro>
 </robot>

Commit message: Add new macro "PLAIN_LINK"

File: src/motion/manipulator/urdf/arcsys2.xacro (robot description, xacro)
@@ -13,13 +13,9 @@
   <xacro:property name="arm1_length" value="0.5"/>
   <xacro:property name="arm2_length" value="0.5"/>
-  <xacro:LINK name="world">
-    <origin xyz="0 0 0" />
-  </xacro:LINK>
+  <xacro:PLAIN_LINK name="world"/>
   <xacro:JOINT parent="world" child="shaft" type="prismatic" y="1" lower="-5.0" upper="5.0">
     <origin xyz="0 0 ${shaft_height/2}"/>
   </xacro:JOINT>
-  <xacro:LINK name="shaft" width="${shaft_thickness}" length="${shaft_thickness}" height="${shaft_height}" color="red">
-    <origin xyz="0 0 0"/>
-  </xacro:LINK>
+  <xacro:PLAIN_LINK name="shaft" length="${shaft_thickness}" width="${shaft_thickness}" height="${shaft_height}" color="red"/>
   <xacro:JOINT parent="shaft" child="arm0" type="prismatic" z="1" lower="-0.5" upper="0.5">
     <origin xyz="${shaft_thickness/2} 0 ${shaft_height/4}"/>
@@ -28,14 +24,8 @@
     <origin xyz="${arm0_length/2} 0 0"/>
   </xacro:LINK>
-  <!--xacro:JOINT parent="arm0" child="arm1" type="revolute" z="1">
-    <origin xyz="${arm0_length} 0 0"/>
-  </xacro:JOINT-->
   <xacro:SCARA_JOINT parent="arm0" child="arm1" parent_length="${arm0_length}"/>
   <xacro:LINK name="arm1" width="${arm_width}" length="${arm1_length}" height="${arm_height}" color="blue">
     <origin xyz="${arm1_length/2} 0 0"/>
   </xacro:LINK>
-  <!--xacro:JOINT parent="arm1" child="arm2" type="revolute" z="1">
-    <origin xyz="${arm1_length} 0 0"/>
-  </xacro:JOINT-->
   <xacro:SCARA_JOINT parent="arm1" child="arm2" parent_length="${arm1_length}"/>
   <xacro:LINK name="arm2" width="${arm_width}" length="${arm2_length}" height="${arm_height}" color="red">
@@ -46,4 +36,15 @@
       <visual>
         <xacro:insert_block name="origin"/>
+        <geometry>
+          <box size="${length} ${width} ${height}"/>
+        </geometry>
+        <material name="${color}"/>
+      </visual>
+    </link>
+  </xacro:macro>
+  <xacro:macro name="PLAIN_LINK" params="name width:=0 length:=0 height:=0 color:=white">
+    <link name="${name}">
+      <origin xyz="0 0 0"/>
+      <visual>
         <geometry>
           <box size="${length} ${width} ${height}"/>

Commit message: Add new macro "SCARA_LINK"

File: src/motion/manipulator/urdf/arcsys2.xacro (robot description, xacro)
@@ -21,15 +21,18 @@
     <origin xyz="${shaft_thickness/2} 0 ${shaft_height/4}"/>
   </xacro:JOINT>
-  <xacro:LINK name="arm0" width="${arm_width}" length="${arm0_length}" height="${arm_height}" color="green">
+  <!--xacro:LINK name="arm0" width="${arm_width}" length="${arm0_length}" height="${arm_height}" color="green">
     <origin xyz="${arm0_length/2} 0 0"/>
-  </xacro:LINK>
+  </xacro:LINK-->
+  <xacro:SCARA_LINK name="arm0" width="${arm_width}" length="${arm0_length}" height="${arm_height}" color="green"/>
   <xacro:SCARA_JOINT parent="arm0" child="arm1" parent_length="${arm0_length}"/>
-  <xacro:LINK name="arm1" width="${arm_width}" length="${arm1_length}" height="${arm_height}" color="blue">
+  <!--xacro:LINK name="arm1" width="${arm_width}" length="${arm1_length}" height="${arm_height}" color="blue">
     <origin xyz="${arm1_length/2} 0 0"/>
-  </xacro:LINK>
+  </xacro:LINK-->
+  <xacro:SCARA_LINK name="arm1" width="${arm_width}" length="${arm1_length}" height="${arm_height}" color="blue"/>
   <xacro:SCARA_JOINT parent="arm1" child="arm2" parent_length="${arm1_length}"/>
-  <xacro:LINK name="arm2" width="${arm_width}" length="${arm2_length}" height="${arm_height}" color="red">
+  <!--xacro:LINK name="arm2" width="${arm_width}" length="${arm2_length}" height="${arm_height}" color="red">
     <origin xyz="${arm2_length/2} 0 0"/>
-  </xacro:LINK>
+  </xacro:LINK-->
+  <xacro:SCARA_LINK name="arm2" width="${arm_width}" length="${arm2_length}" height="${arm_height}" color="red"/>
   <xacro:macro name="LINK" params="name width:=0 length:=0 height:=0 color:=white *origin">
     <link name="${name}">
@@ -47,4 +50,15 @@
       <origin xyz="0 0 0"/>
       <visual>
+        <geometry>
+          <box size="${length} ${width} ${height}"/>
+        </geometry>
+        <material name="${color}"/>
+      </visual>
+    </link>
+  </xacro:macro>
+  <xacro:macro name="SCARA_LINK" params="name width:=0 length:=0 height:=0 color:=white">
+    <link name="${name}">
+      <visual>
+        <origin xyz="${length/2} 0 0"/>
         <geometry>
           <box size="${length} ${width} ${height}"/>

Commit message: Delete unused macro and comment

File: src/motion/manipulator/urdf/arcsys2.xacro (robot description, xacro)
@@ -21,29 +21,9 @@
     <origin xyz="${shaft_thickness/2} 0 ${shaft_height/4}"/>
   </xacro:JOINT>
-  <!--xacro:LINK name="arm0" width="${arm_width}" length="${arm0_length}" height="${arm_height}" color="green">
-    <origin xyz="${arm0_length/2} 0 0"/>
-  </xacro:LINK-->
   <xacro:SCARA_LINK name="arm0" width="${arm_width}" length="${arm0_length}" height="${arm_height}" color="green"/>
   <xacro:SCARA_JOINT parent="arm0" child="arm1" parent_length="${arm0_length}"/>
-  <!--xacro:LINK name="arm1" width="${arm_width}" length="${arm1_length}" height="${arm_height}" color="blue">
-    <origin xyz="${arm1_length/2} 0 0"/>
-  </xacro:LINK-->
   <xacro:SCARA_LINK name="arm1" width="${arm_width}" length="${arm1_length}" height="${arm_height}" color="blue"/>
   <xacro:SCARA_JOINT parent="arm1" child="arm2" parent_length="${arm1_length}"/>
-  <!--xacro:LINK name="arm2" width="${arm_width}" length="${arm2_length}" height="${arm_height}" color="red">
-    <origin xyz="${arm2_length/2} 0 0"/>
-  </xacro:LINK-->
   <xacro:SCARA_LINK name="arm2" width="${arm_width}" length="${arm2_length}" height="${arm_height}" color="red"/>
-  <xacro:macro name="LINK" params="name width:=0 length:=0 height:=0 color:=white *origin">
-    <link name="${name}">
-      <visual>
-        <xacro:insert_block name="origin"/>
-        <geometry>
-          <box size="${length} ${width} ${height}"/>
-        </geometry>
-        <material name="${color}"/>
-      </visual>
-    </link>
-  </xacro:macro>
   <xacro:macro name="PLAIN_LINK" params="name width:=0 length:=0 height:=0 color:=white">
     <link name="${name}">

Commit message: Change naming macro of joint

File: src/motion/manipulator/urdf/arcsys2.xacro (robot description, xacro)
@@ -14,15 +14,15 @@
   <xacro:property name="arm2_length" value="0.5"/>
   <xacro:PLAIN_LINK name="world"/>
-  <xacro:JOINT parent="world" child="shaft" type="prismatic" y="1" lower="-5.0" upper="5.0">
+  <xacro:JOINT name="world->shaft" type="prismatic" y="1" lower="-5.0" upper="5.0">
     <origin xyz="0 0 ${shaft_height/2}"/>
   </xacro:JOINT>
   <xacro:PLAIN_LINK name="shaft" length="${shaft_thickness}" width="${shaft_thickness}" height="${shaft_height}" color="red"/>
-  <xacro:JOINT parent="shaft" child="arm0" type="prismatic" z="1" lower="-0.5" upper="0.5">
+  <xacro:JOINT name="shaft->arm0" type="prismatic" z="1" lower="-0.5" upper="0.5">
     <origin xyz="${shaft_thickness/2} 0 ${shaft_height/4}"/>
   </xacro:JOINT>
   <xacro:SCARA_LINK name="arm0" width="${arm_width}" length="${arm0_length}" height="${arm_height}" color="green"/>
-  <xacro:SCARA_JOINT parent="arm0" child="arm1" parent_length="${arm0_length}"/>
+  <xacro:SCARA_JOINT name="arm0->arm1" parent_length="${arm0_length}"/>
   <xacro:SCARA_LINK name="arm1" width="${arm_width}" length="${arm1_length}" height="${arm_height}" color="blue"/>
-  <xacro:SCARA_JOINT parent="arm1" child="arm2" parent_length="${arm1_length}"/>
+  <xacro:SCARA_JOINT name="arm1->arm2" parent_length="${arm1_length}"/>
   <xacro:SCARA_LINK name="arm2" width="${arm_width}" length="${arm2_length}" height="${arm_height}" color="red"/>
   <xacro:macro name="PLAIN_LINK" params="name width:=0 length:=0 height:=0 color:=white">
@@ -48,6 +48,6 @@
     </link>
   </xacro:macro>
-  <xacro:macro name="JOINT" params="parent child type x:=0 y:=0 z:=0 lower:=${-pi/2} upper:=${pi/2} *origin">
-    <joint name="${parent}->${child}" type="${type}">
+  <xacro:macro name="JOINT" params="name type x:=0 y:=0 z:=0 lower:=${-pi/2} upper:=${pi/2} *origin">
+    <joint name="${name}" type="${type}">
       <xacro:insert_block name="origin"/>
       <parent link="${parent}"/>
@@ -57,6 +57,6 @@
     </joint>
   </xacro:macro>
-  <xacro:macro name="SCARA_JOINT" params="parent child parent_length lower:=${-pi/2} upper:=${pi/2}">
-    <joint name="${parent}->${child}" type="revolute">
+  <xacro:macro name="SCARA_JOINT" params="parent_length lower:=${-pi/2} upper:=${pi/2}">
+    <joint name="${name}" type="revolute">
       <origin xyz="${parent_length} 0 0"/>
       <parent link="${parent}"/>

Commit message: Change macro JOINT to PRISMATIC_JOINT
今回のロボットには PRISMATIC か SCARAなジョイントしか登場しないと
予想されるため汎用の JOINT マクロは廃止

File: src/motion/manipulator/urdf/arcsys2.xacro (robot description, xacro)
@@ -14,9 +14,9 @@
   <xacro:property name="arm2_length" value="0.5"/>
   <xacro:PLAIN_LINK name="world"/>
-  <xacro:JOINT name="world->shaft" type="prismatic" y="1" lower="-5.0" upper="5.0">
+  <xacro:PRISMATIC_JOINT name="world->shaft" y="1" lower="-5.0" upper="5.0">
     <origin xyz="0 0 ${shaft_height/2}"/>
   </xacro:JOINT>
   <xacro:PLAIN_LINK name="shaft" length="${shaft_thickness}" width="${shaft_thickness}" height="${shaft_height}" color="red"/>
-  <xacro:JOINT name="shaft->arm0" type="prismatic" z="1" lower="-0.5" upper="0.5">
+  <xacro:PRISMATIC_JOINT name="shaft->arm0" z="1" lower="-0.5" upper="0.5">
     <origin xyz="${shaft_thickness/2} 0 ${shaft_height/4}"/>
   </xacro:JOINT>
@@ -48,6 +48,6 @@
     </link>
   </xacro:macro>
-  <xacro:macro name="JOINT" params="name type x:=0 y:=0 z:=0 lower:=${-pi/2} upper:=${pi/2} *origin">
-    <joint name="${name}" type="${type}">
+  <xacro:macro name="PRISMATIC_JOINT" params="name x:=0 y:=0 z:=0 lower:=${-pi/2} upper:=${pi/2} *origin">
+    <joint name="${name}" type="prismatic">
       <xacro:insert_block name="origin"/>
       <parent link="${parent}"/>

Commit message: Add new macro "default_size"
長さにシミュレーション上特に意味は無いが
ビジュアル的に可視であってほしいリンクのサイズに
0.1 がとりあえずの値として設定されており
これをプロパティに指定するマクロが複数あったため
「デフォルト値」という形で統一

File: src/motion/manipulator/urdf/arcsys2.xacro (robot description, xacro)
@@ -6,25 +6,26 @@
   <material name="blue">  <color rgba="${  0/255} ${  0/255} ${255/255} 1.0" /> </material>
   <xacro:property name="pi" value="3.1415"/>
+  <xacro:property name="default_size" value="0.1"/>
   <xacro:property name="shaft_height" value="2.0"/>
-  <xacro:property name="shaft_thickness" value="0.1"/>
-  <xacro:property name="arm_width" value="0.1"/>
-  <xacro:property name="arm_height" value="${arm_width}"/>
+  <!--xacro:property name="shaft_thickness" value="0.1"/-->
+  <!--xacro:property name="arm_width" value="0.1"/-->
+  <!--xacro:property name="arm_height" value="${arm_width}"/-->
   <xacro:property name="arm0_length" value="0.1"/>
   <xacro:property name="arm1_length" value="0.5"/>
   <xacro:property name="arm2_length" value="0.5"/>
   <xacro:PLAIN_LINK name="world"/>
-  <xacro:PRISMATIC_JOINT name="world->shaft" y="1" lower="-5.0" upper="5.0">
+  <xacro:PRISMATIC_JOINT parent="world" child="shaft" y="1" lower="-5.0" upper="5.0">
     <origin xyz="0 0 ${shaft_height/2}"/>
-  </xacro:JOINT>
-  <xacro:PLAIN_LINK name="shaft" length="${shaft_thickness}" width="${shaft_thickness}" height="${shaft_height}" color="red"/>
-  <xacro:PRISMATIC_JOINT name="shaft->arm0" z="1" lower="-0.5" upper="0.5">
-    <origin xyz="${shaft_thickness/2} 0 ${shaft_height/4}"/>
-  </xacro:JOINT>
-  <xacro:SCARA_LINK name="arm0" width="${arm_width}" length="${arm0_length}" height="${arm_height}" color="green"/>
-  <xacro:SCARA_JOINT name="arm0->arm1" parent_length="${arm0_length}"/>
-  <xacro:SCARA_LINK name="arm1" width="${arm_width}" length="${arm1_length}" height="${arm_height}" color="blue"/>
-  <xacro:SCARA_JOINT name="arm1->arm2" parent_length="${arm1_length}"/>
-  <xacro:SCARA_LINK name="arm2" width="${arm_width}" length="${arm2_length}" height="${arm_height}" color="red"/>
-  <xacro:macro name="PLAIN_LINK" params="name width:=0 length:=0 height:=0 color:=white">
+  </xacro:PRISMATIC_JOINT>
+  <xacro:PLAIN_LINK name="shaft" height="${shaft_height}" color="red"/>
+  <xacro:PRISMATIC_JOINT parent="shaft" child="arm0" z="1" lower="-0.5" upper="0.5">
+    <origin xyz="${default_size/2} 0 ${shaft_height/4}"/>
+  </xacro:PRISMATIC_JOINT>
+  <xacro:SCARA_LINK name="arm0" length="${arm0_length}" color="green"/>
+  <xacro:SCARA_JOINT parent="arm0" child="arm1" parent_length="${arm0_length}"/>
+  <xacro:SCARA_LINK name="arm1" length="${arm1_length}" color="blue"/>
+  <xacro:SCARA_JOINT parent="arm1" child="arm2" parent_length="${arm1_length}"/>
+  <xacro:SCARA_LINK name="arm2" length="${arm2_length}" color="red"/>
+  <xacro:macro name="PLAIN_LINK" params="name width:=${default_size} length:=${default_size} height:=${default_size} color:=white">
     <link name="${name}">
       <origin xyz="0 0 0"/>
@@ -37,5 +38,5 @@
     </link>
   </xacro:macro>
-  <xacro:macro name="SCARA_LINK" params="name width:=0 length:=0 height:=0 color:=white">
+  <xacro:macro name="SCARA_LINK" params="name width:=${default_size} length:=${default_size} height:=${default_size} color:=white">
     <link name="${name}">
       <visual>
@@ -48,6 +49,6 @@
     </link>
   </xacro:macro>
-  <xacro:macro name="PRISMATIC_JOINT" params="name x:=0 y:=0 z:=0 lower:=${-pi/2} upper:=${pi/2} *origin">
-    <joint name="${name}" type="prismatic">
+  <xacro:macro name="PRISMATIC_JOINT" params="parent child x:=0 y:=0 z:=0 lower:=${-pi/2} upper:=${pi/2} *origin">
+    <joint name="${parent}->${child}" type="prismatic">
       <xacro:insert_block name="origin"/>
       <parent link="${parent}"/>
@@ -57,6 +58,6 @@
     </joint>
   </xacro:macro>
-  <xacro:macro name="SCARA_JOINT" params="parent_length lower:=${-pi/2} upper:=${pi/2}">
-    <joint name="${name}" type="revolute">
+  <xacro:macro name="SCARA_JOINT" params="parent child parent_length lower:=${-pi/2} upper:=${pi/2}">
+    <joint name="${parent}->${child}" type="revolute">
       <origin xyz="${parent_length} 0 0"/>
       <parent link="${parent}"/>

Commit message: Clean up

File: src/motion/manipulator/urdf/arcsys2.xacro (robot description, xacro)
@@ -5,13 +5,13 @@
   <material name="green"> <color rgba="${  0/255} ${255/255} ${  0/255} 1.0" /> </material>
   <material name="blue">  <color rgba="${  0/255} ${  0/255} ${255/255} 1.0" /> </material>
-  <xacro:property name="pi" value="3.1415"/>
+<!-- Property -->
+  <xacro:property name="pi" value="3.1415926535897931" />
   <xacro:property name="default_size" value="0.1"/>
-  <xacro:property name="shaft_height" value="2.0"/>
-  <!--xacro:property name="shaft_thickness" value="0.1"/-->
-  <!--xacro:property name="arm_width" value="0.1"/-->
-  <!--xacro:property name="arm_height" value="${arm_width}"/-->
-  <xacro:property name="arm0_length" value="0.1"/>
-  <xacro:property name="arm1_length" value="0.5"/>
-  <xacro:property name="arm2_length" value="0.5"/>
+  <xacro:property name="shaft_height"    value="2.0"/>
+  <xacro:property name="arm0_length"     value="0.1"/>
+  <xacro:property name="arm1_length"     value="0.5"/>
+  <xacro:property name="arm2_length"     value="0.5"/>
+  <xacro:property name="effector_length" value="0.5"/>
+<!-- LINK and JOINT -->
   <xacro:PLAIN_LINK name="world"/>
   <xacro:PRISMATIC_JOINT parent="world" child="shaft" y="1" lower="-5.0" upper="5.0">
@@ -27,4 +27,7 @@
   <xacro:SCARA_JOINT parent="arm1" child="arm2" parent_length="${arm1_length}"/>
   <xacro:SCARA_LINK name="arm2" length="${arm2_length}" color="red"/>
+  <xacro:SCARA_JOINT parent="arm2" child="effector" parent_length="${arm2_length}"/>
+  <xacro:SCARA_LINK name="effector" length="${effector_length}" color="green"/>
+<!-- Macro Definition -->
   <xacro:macro name="PLAIN_LINK" params="name width:=${default_size} length:=${default_size} height:=${default_size} color:=white">
     <link name="${name}">
