Commit message: Add collision to each links

File: src/motion/arcsys2_description/urdf/arcsys2.xacro (robot description, xacro)
@@ -39,4 +39,9 @@
         <material name="${color}"/>
       </visual>
+      <collision>
+        <geometry>
+          <box size="${length} ${width} ${height}"/>
+        </geometry>
+      </collision>
     </link>
   </xacro:macro>
@@ -50,4 +55,9 @@
         <material name="${color}"/>
       </visual>
+      <collision>
+        <geometry>
+          <box size="${length} ${width} ${height}"/>
+        </geometry>
+      </collision>
     </link>
   </xacro:macro>

Commit message: Change prefix to "_" from "->"

File: src/motion/arcsys2_description/urdf/arcsys2.xacro (robot description, xacro)
@@ -63,5 +63,5 @@
   </xacro:macro>
   <xacro:macro name="PRISMATIC_JOINT" params="parent child x:=0 y:=0 z:=0 lower:=${-pi/2} upper:=${pi/2} *origin">
-    <joint name="${parent}->${child}" type="prismatic">
+    <joint name="${parent}_${child}" type="prismatic">
       <xacro:insert_block name="origin"/>
       <parent link="${parent}"/>
@@ -72,5 +72,5 @@
   </xacro:macro>
   <xacro:macro name="SCARA_JOINT" params="parent child parent_length lower:=${-pi/2} upper:=${pi/2}">
-    <joint name="${parent}->${child}" type="revolute">
+    <joint name="${parent}_${child}" type="revolute">
       <origin xyz="${parent_length} 0 0"/>
       <parent link="${parent}"/>

Commit message: Change prefix to "_to_" from "_"

File: src/motion/arcsys2_description/urdf/arcsys2.xacro (robot description, xacro)
@@ -63,5 +63,5 @@
   </xacro:macro>
   <xacro:macro name="PRISMATIC_JOINT" params="parent child x:=0 y:=0 z:=0 lower:=${-pi/2} upper:=${pi/2} *origin">
-    <joint name="${parent}_${child}" type="prismatic">
+    <joint name="${parent}_to_${child}" type="prismatic">
       <xacro:insert_block name="origin"/>
       <parent link="${parent}"/>
@@ -72,5 +72,5 @@
   </xacro:macro>
   <xacro:macro name="SCARA_JOINT" params="parent child parent_length lower:=${-pi/2} upper:=${pi/2}">
-    <joint name="${parent}_${child}" type="revolute">
+    <joint name="${parent}_to_${child}" type="revolute">
       <origin xyz="${parent_length} 0 0"/>
       <parent link="${parent}"/>

Commit message: Change base_link to rail from world

File: src/motion/arcsys2_description/urdf/arcsys2.xacro (robot description, xacro)
@@ -8,4 +8,5 @@
   <xacro:property name="pi" value="3.1415926535897931" />
   <xacro:property name="default_size" value="0.1"/>
+  <xacro:property name="rail_length"     value="10.0" />
   <xacro:property name="shaft_height"    value="2.0"/>
   <xacro:property name="arm0_length"     value="0.1"/>
@@ -14,6 +15,6 @@
   <xacro:property name="effector_length" value="0.5"/>
 <!-- LINK and JOINT -->
-  <xacro:PLAIN_LINK name="world"/>
-  <xacro:PRISMATIC_JOINT parent="world" child="shaft" y="1" lower="-5.0" upper="5.0">
+  <xacro:PLAIN_LINK width="${rail_length}" name="rail"/>
+  <xacro:PRISMATIC_JOINT parent="rail" child="shaft" y="1" lower="${-1*rail_length/2}" upper="${rail_length/2}">
     <origin xyz="0 0 ${shaft_height/2}"/>
   </xacro:PRISMATIC_JOINT>

Commit message: Add joint that do not actually exist for dof test
5自由度以下での使用に適していないのなら
現実には存在しない手首ジョイントを加えて6自由度とすればいいのではないか

目標Poseにひねりの要素を与えなければあっても無くても変わらないはず

File: src/motion/arcsys2_description/urdf/arcsys2.xacro (robot description, xacro)
@@ -28,6 +28,8 @@
   <xacro:SCARA_JOINT parent="arm1" child="arm2" parent_length="${arm1_length}"/>
   <xacro:SCARA_LINK name="arm2" length="${arm2_length}" color="red"/>
-  <xacro:SCARA_JOINT parent="arm2" child="effector" parent_length="${arm2_length}"/>
-  <xacro:SCARA_LINK name="effector" length="${effector_length}" color="green"/>
+  <xacro:SCARA_JOINT parent="arm2" child="effector_base" parent_length="${arm2_length}"/>
+  <xacro:SCARA_LINK name="effector_base" length="${effector_length/2}" color="green"/>
+  <xacro:WRIST_JOINT parent="effector_base" child="effector_end" parent_length="${effector_length/2}" />
+  <xacro:SCARA_LINK name="effector_end" length="${effector_length/2}" color="blue" />
 <!-- Macro Definition -->
   <xacro:macro name="PLAIN_LINK" params="name width:=${default_size} length:=${default_size} height:=${default_size} color:=white">
@@ -81,3 +83,12 @@
     </joint>
   </xacro:macro>
+  <xacro:macro name="WRIST_JOINT" params="parent child parent_length lower:=${-pi/2} upper:=${pi/2}">
+    <joint name="${parent}_to_${child}" type="revolute">
+      <origin xyz="${parent_length} 0 0"/>
+      <parent link="${parent}"/>
+      <child link="${child}"/>
+      <axis xyz="1 0 0"/>
+      <limit lower="${lower}" upper="${upper}" effort="1" velocity="1"/>
+    </joint>
+  </xacro:macro>
 </robot>

Commit message: Add transmission element to arcsys2.xacro

File: src/motion/arcsys2_description/urdf/arcsys2.xacro (robot description, xacro)
@@ -14,4 +14,6 @@
   <xacro:property name="arm2_length"     value="0.5"/>
   <xacro:property name="effector_length" value="0.5"/>
+  <xacro:property name="default_hardware_interface"
+                 value="hardware_interface/PositionJointInterface" />
 <!-- LINK and JOINT -->
   <xacro:PLAIN_LINK width="${rail_length}" name="rail"/>
@@ -65,6 +67,6 @@
     </link>
   </xacro:macro>
-  <xacro:macro name="PRISMATIC_JOINT" params="parent child x:=0 y:=0 z:=0 lower:=${-pi/2} upper:=${pi/2} *origin">
-    <joint name="${parent}_to_${child}" type="prismatic">
+  <xacro:macro name="PRISMATIC_JOINT" params="parent child x:=0 y:=0 z:=0 lower:=${-pi/2} upper:=${pi/2} *origin reduction:=1.0 hardware_interface:=${default_hardware_interface}">
+    <joint name="${parent}_to_${child}_joint" type="prismatic">
       <xacro:insert_block name="origin"/>
       <parent link="${parent}"/>
@@ -73,7 +75,17 @@
       <limit lower="${lower}" upper="${upper}" effort="1" velocity="1"/>
     </joint>
+    <transmission name="${parent}_to_${child}_transmission">
+      <type>transmission_interface/SimpleTransmission</type>
+      <actuator name="${parent}_to_${child}_actuator">
+        <mechanicalReduction>${reduction}</mechanicalReduction>
+        <hardwareInterface>${default_hardware_interface}</hardwareInterface>
+      </actuator>
+      <joint name="${parent}_to_${child}_joint">
+        <hardwareInterface>${default_hardware_interface}</hardwareInterface>
+      </joint>
+    </transmission>
   </xacro:macro>
-  <xacro:macro name="SCARA_JOINT" params="parent child parent_length lower:=${-pi/2} upper:=${pi/2}">
-    <joint name="${parent}_to_${child}" type="revolute">
+  <xacro:macro name="SCARA_JOINT" params="parent child parent_length lower:=${-pi/2} upper:=${pi/2} reduction:=1.0 hardware_interface:=${default_hardware_interface}">
+    <joint name="${parent}_to_${child}_joint" type="revolute">
       <origin xyz="${parent_length} 0 0"/>
       <parent link="${parent}"/>
@@ -82,7 +94,17 @@
       <limit lower="${lower}" upper="${upper}" effort="1" velocity="1"/>
     </joint>
+    <transmission name="${parent}_to_${child}_transmission">
+      <type>transmission_interface/SimpleTransmission</type>
+      <actuator name="${parent}_to_${child}_actuator">
+        <mechanicalReduction>${reduction}</mechanicalReduction>
+        <hardwareInterface>${default_hardware_interface}</hardwareInterface>
+      </actuator>
+      <joint name="${parent}_to_${child}_joint">
+        <hardwareInterface>${default_hardware_interface}</hardwareInterface>
+      </joint>
+    </transmission>
   </xacro:macro>
-  <xacro:macro name="WRIST_JOINT" params="parent child parent_length lower:=${-pi/2} upper:=${pi/2}">
-    <joint name="${parent}_to_${child}" type="revolute">
+  <xacro:macro name="WRIST_JOINT" params="parent child parent_length lower:=${-pi/2} upper:=${pi/2} reduction:=1.0 hardware_interface:=${default_hardware_interface}">
+    <joint name="${parent}_to_${child}_joint" type="revolute">
       <origin xyz="${parent_length} 0 0"/>
       <parent link="${parent}"/>
@@ -91,4 +113,14 @@
       <limit lower="${lower}" upper="${upper}" effort="1" velocity="1"/>
     </joint>
+    <transmission name="${parent}_to_${child}_transmission">
+      <type>transmission_interface/SimpleTransmission</type>
+      <actuator name="${parent}_to_${child}_actuator">
+        <mechanicalReduction>${reduction}</mechanicalReduction>
+        <hardwareInterface>${default_hardware_interface}</hardwareInterface>
+      </actuator>
+      <joint name="${parent}_to_${child}_joint">
+        <hardwareInterface>${default_hardware_interface}</hardwareInterface>
+      </joint>
+    </transmission>
   </xacro:macro>
 </robot>
