Commit message: Add fixed joint xacro:macro

File: src/arcsys2_description/urdf/arcsys2.xacro (robot description, xacro)
@@ -67,4 +67,11 @@
     </link>
   </xacro:macro>
+  <xacro:macro name="FIXED_JOINT" params="parent child *origin">
+    <joint name="${parent}_to_${child}_joint" type="fixed">
+      <xacro:insert_block name="origin"/>
+      <parent link="${parent}"/>
+      <child link="${child}"/>
+    </joint>
+  </xacro:macro>
   <xacro:macro name="PRISMATIC_JOINT" params="parent child x:=0 y:=0 z:=0 lower:=${-pi/2} upper:=${pi/2} *origin reduction:=1.0 hardware_interface:=${default_hardware_interface}">
     <joint name="${parent}_to_${child}_joint" type="prismatic">

Commit message: Add link "kinect"

File: src/arcsys2_description/urdf/arcsys2.xacro (robot description, xacro)
@@ -34,4 +34,8 @@
   <xacro:WRIST_JOINT parent="effector_base" child="effector_end" parent_length="${effector_length/2}" />
   <xacro:SCARA_LINK name="effector_end" length="${effector_length/2}" color="blue" />
+  <xacro:FIXED_JOINT parent="shaft" child="kinect">
+    <origin xyz="0 0 ${shaft_height/2}" />
+  </xacro:FIXED_JOINT>
+  <xacro:PLAIN_LINK name="kinect" color="green" />
 <!-- Macro Definition -->
   <xacro:macro name="PLAIN_LINK" params="name width:=${default_size} length:=${default_size} height:=${default_size} color:=white">

Commit message: Cleanup unneeded code for gazebo

File: src/arcsys2_description/urdf/arcsys2.xacro (robot description, xacro)
@@ -13,7 +13,5 @@
   <xacro:property name="arm1_length"     value="0.5"/>
   <xacro:property name="arm2_length"     value="0.5"/>
-  <xacro:property name="effector_length" value="0.5"/>
-  <xacro:property name="default_hardware_interface"
-                 value="hardware_interface/PositionJointInterface" />
+  <xacro:property name="eff_length" value="0.5"/>
 <!-- LINK and JOINT -->
   <xacro:PLAIN_LINK width="${rail_length}" name="rail"/>
@@ -31,7 +29,7 @@
   <xacro:SCARA_LINK name="arm2" length="${arm2_length}" color="red"/>
   <xacro:SCARA_JOINT parent="arm2" child="effector_base" parent_length="${arm2_length}"/>
-  <xacro:SCARA_LINK name="effector_base" length="${effector_length/2}" color="green"/>
-  <xacro:WRIST_JOINT parent="effector_base" child="effector_end" parent_length="${effector_length/2}" />
-  <xacro:SCARA_LINK name="effector_end" length="${effector_length/2}" color="blue" />
+  <xacro:SCARA_LINK name="effector_base" length="${eff_length/2}" color="green"/>
+  <xacro:WRIST_JOINT parent="effector_base" child="effector_end" parent_length="${eff_length/2}" />
+  <xacro:SCARA_LINK name="effector_end" length="${eff_length/2}" color="blue" />
   <xacro:FIXED_JOINT parent="shaft" child="kinect">
     <origin xyz="0 0 ${shaft_height/2}" />
@@ -78,5 +76,5 @@
     </joint>
   </xacro:macro>
-  <xacro:macro name="PRISMATIC_JOINT" params="parent child x:=0 y:=0 z:=0 lower:=${-pi/2} upper:=${pi/2} *origin reduction:=1.0 hardware_interface:=${default_hardware_interface}">
+  <xacro:macro name="PRISMATIC_JOINT" params="parent child x:=0 y:=0 z:=0 lower:=-1 upper:=1 *origin">
     <joint name="${parent}_to_${child}_joint" type="prismatic">
       <xacro:insert_block name="origin"/>
@@ -86,16 +84,6 @@
       <limit lower="${lower}" upper="${upper}" effort="1" velocity="1"/>
     </joint>
-    <transmission name="${parent}_to_${child}_transmission">
-      <type>transmission_interface/SimpleTransmission</type>
-      <actuator name="${parent}_to_${child}_actuator">
-        <mechanicalReduction>${reduction}</mechanicalReduction>
-        <hardwareInterface>${default_hardware_interface}</hardwareInterface>
-      </actuator>
-      <joint name="${parent}_to_${child}_joint">
-        <hardwareInterface>${default_hardware_interface}</hardwareInterface>
-      </joint>
-    </transmission>
   </xacro:macro>
-  <xacro:macro name="SCARA_JOINT" params="parent child parent_length lower:=${-pi/2} upper:=${pi/2} reduction:=1.0 hardware_interface:=${default_hardware_interface}">
+  <xacro:macro name="SCARA_JOINT" params="parent child parent_length lower:=${-pi/2}">
     <joint name="${parent}_to_${child}_joint" type="revolute">
       <origin xyz="${parent_length} 0 0"/>
@@ -105,16 +93,6 @@
       <limit lower="${lower}" upper="${upper}" effort="1" velocity="1"/>
     </joint>
-    <transmission name="${parent}_to_${child}_transmission">
-      <type>transmission_interface/SimpleTransmission</type>
-      <actuator name="${parent}_to_${child}_actuator">
-        <mechanicalReduction>${reduction}</mechanicalReduction>
-        <hardwareInterface>${default_hardware_interface}</hardwareInterface>
-      </actuator>
-      <joint name="${parent}_to_${child}_joint">
-        <hardwareInterface>${default_hardware_interface}</hardwareInterface>
-      </joint>
-    </transmission>
   </xacro:macro>
-  <xacro:macro name="WRIST_JOINT" params="parent child parent_length lower:=${-pi/2} upper:=${pi/2} reduction:=1.0 hardware_interface:=${default_hardware_interface}">
+  <xacro:macro name="WRIST_JOINT" params="parent child parent_length lower:=${-pi/2} upper:=${pi/2}">
     <joint name="${parent}_to_${child}_joint" type="revolute">
       <origin xyz="${parent_length} 0 0"/>
@@ -124,14 +102,4 @@
       <limit lower="${lower}" upper="${upper}" effort="1" velocity="1"/>
     </joint>
-    <transmission name="${parent}_to_${child}_transmission">
-      <type>transmission_interface/SimpleTransmission</type>
-      <actuator name="${parent}_to_${child}_actuator">
-        <mechanicalReduction>${reduction}</mechanicalReduction>
-        <hardwareInterface>${default_hardware_interface}</hardwareInterface>
-      </actuator>
-      <joint name="${parent}_to_${child}_joint">
-        <hardwareInterface>${default_hardware_interface}</hardwareInterface>
-      </joint>
-    </transmission>
   </xacro:macro>
 </robot>

Commit message: Cleanup

File: src/arcsys2_description/urdf/arcsys2.xacro (robot description, xacro)
@@ -7,13 +7,13 @@
 <!-- Property -->
   <xacro:property name="pi" value="3.1415926535897931" />
-  <xacro:property name="default_size" value="0.1"/>
-  <xacro:property name="rail_length"     value="10.0" />
-  <xacro:property name="shaft_height"    value="2.0"/>
-  <xacro:property name="arm0_length"     value="0.1"/>
-  <xacro:property name="arm1_length"     value="0.5"/>
-  <xacro:property name="arm2_length"     value="0.5"/>
-  <xacro:property name="eff_length" value="0.5"/>
+  <xacro:property name="default_size" value="0.1" />
+  <xacro:property name="rail_length"  value="10.0" />
+  <xacro:property name="shaft_height" value="2.0" />
+  <xacro:property name="arm0_length"  value="0.1" />
+  <xacro:property name="arm1_length"  value="0.5" />
+  <xacro:property name="arm2_length"  value="0.5" />
+  <xacro:property name="eff_length"   value="0.5" />
 <!-- LINK and JOINT -->
-  <xacro:PLAIN_LINK width="${rail_length}" name="rail"/>
+  <xacro:PLAIN_LINK name="rail" width="${rail_length}" />
   <xacro:PRISMATIC_JOINT parent="rail" child="shaft" y="1" lower="${-1*rail_length/2}" upper="${rail_length/2}">
     <origin xyz="0 0 ${shaft_height/2}"/>

Commit message: Update to actual size

File: src/arcsys2_description/urdf/arcsys2.xacro (robot description, xacro)
@@ -8,13 +8,13 @@
   <xacro:property name="pi" value="3.1415926535897931" />
   <xacro:property name="default_size" value="0.1" />
-  <xacro:property name="rail_length"  value="10.0" />
-  <xacro:property name="shaft_height" value="2.0" />
-  <xacro:property name="arm0_length"  value="0.1" />
-  <xacro:property name="arm1_length"  value="0.5" />
-  <xacro:property name="arm2_length"  value="0.5" />
-  <xacro:property name="eff_length"   value="0.5" />
+  <xacro:property name="rail_length"  value="3.600" /> <!-- OK? -->
+  <xacro:property name="shaft_height" value="2.000" />
+  <xacro:property name="arm0_length"  value="0.100" />
+  <xacro:property name="arm1_length"  value="0.216" /> <!-- OK? -->
+  <xacro:property name="arm2_length"  value="0.199" /> <!-- OK? -->
+  <xacro:property name="eff_length"   value="0.225" /> <!-- OK? -->
 <!-- LINK and JOINT -->
-  <xacro:PLAIN_LINK name="rail" width="${rail_length}" />
-  <xacro:PRISMATIC_JOINT parent="rail" child="shaft" y="1" lower="${-1*rail_length/2}" upper="${rail_length/2}">
+  <xacro:PLAIN_LINK name="rail" width="${rail_length*2}" />
+  <xacro:PRISMATIC_JOINT parent="rail" child="shaft" y="1" lower="${-1*rail_length}" upper="${rail_length}">
     <origin xyz="0 0 ${shaft_height/2}"/>
   </xacro:PRISMATIC_JOINT>

Commit message: Fix bug

File: src/arcsys2_description/urdf/arcsys2.xacro (robot description, xacro)
@@ -85,5 +85,5 @@
     </joint>
   </xacro:macro>
-  <xacro:macro name="SCARA_JOINT" params="parent child parent_length lower:=${-pi/2}">
+  <xacro:macro name="SCARA_JOINT" params="parent child parent_length lower:=${-pi/2} upper:=${pi/2}">
     <joint name="${parent}_to_${child}_joint" type="revolute">
       <origin xyz="${parent_length} 0 0"/>

Commit message: Set arbitary number for test

File: src/arcsys2_description/urdf/arcsys2.xacro (robot description, xacro)
@@ -9,5 +9,5 @@
   <xacro:property name="default_size" value="0.1" />
   <xacro:property name="rail_length"  value="3.600" /> <!-- OK? -->
-  <xacro:property name="shaft_height" value="2.000" />
+  <xacro:property name="shaft_height" value="1.400" />
   <xacro:property name="arm0_length"  value="0.100" />
   <xacro:property name="arm1_length"  value="0.216" /> <!-- OK? -->
@@ -18,8 +18,11 @@
   <xacro:PRISMATIC_JOINT parent="rail" child="shaft" y="1" lower="${-1*rail_length}" upper="${rail_length}">
     <origin xyz="0 0 ${shaft_height/2}"/>
+    <!-- これのZ座標がキネクトの高度がこれに依存しているので注意 -->
   </xacro:PRISMATIC_JOINT>
   <xacro:PLAIN_LINK name="shaft" height="${shaft_height}" color="red"/>
-  <xacro:PRISMATIC_JOINT parent="shaft" child="arm0" z="1" lower="-0.5" upper="0.5">
+  <xacro:PRISMATIC_JOINT parent="shaft" child="arm0" z="1" lower="-0.2" upper="0.2">
     <origin xyz="${default_size/2} 0 ${shaft_height/4}"/>
+    <!-- ここのdefault_size -> シャフトの奥行き -->
+    <!-- zは初期位置以外の意味は無いと思われる -->
   </xacro:PRISMATIC_JOINT>
   <xacro:SCARA_LINK name="arm0" length="${arm0_length}" color="green"/>
@@ -33,5 +36,5 @@
   <xacro:SCARA_LINK name="effector_end" length="${eff_length/2}" color="blue" />
   <xacro:FIXED_JOINT parent="shaft" child="kinect">
-    <origin xyz="0 0 ${shaft_height/2}" />
+    <origin xyz="0 -0.1 0" />
   </xacro:FIXED_JOINT>
   <xacro:PLAIN_LINK name="kinect" color="green" />

Commit message: Update for debug

File: src/arcsys2_description/urdf/arcsys2.xacro (robot description, xacro)
@@ -34,7 +34,7 @@
   <xacro:SCARA_LINK name="effector_base" length="${eff_length/2}" color="green"/>
   <xacro:WRIST_JOINT parent="effector_base" child="effector_end" parent_length="${eff_length/2}" />
-  <xacro:SCARA_LINK name="effector_end" length="${eff_length/2}" color="blue" />
+  <xacro:SCARA_LINK name="effector_end" length="${eff_length/2}" color="green" />
   <xacro:FIXED_JOINT parent="shaft" child="kinect">
-    <origin xyz="0 -0.1 0" />
+    <origin xyz="0 0.1 0" />
   </xacro:FIXED_JOINT>
   <xacro:PLAIN_LINK name="kinect" color="green" />

Commit message: Fuck Them All

File: src/arcsys2_description/urdf/arcsys2.xacro (robot description, xacro)
@@ -9,6 +9,6 @@
   <xacro:property name="default_size" value="0.1" />
   <xacro:property name="rail_length"  value="3.600" /> <!-- OK? -->
-  <xacro:property name="shaft_height" value="1.400" />
-  <xacro:property name="arm0_length"  value="0.100" />
+  <xacro:property name="shaft_height" value="1.350" />
+  <xacro:property name="arm0_length"  value="0.125" />
   <xacro:property name="arm1_length"  value="0.216" /> <!-- OK? -->
   <xacro:property name="arm2_length"  value="0.199" /> <!-- OK? -->
@@ -36,5 +36,5 @@
   <xacro:SCARA_LINK name="effector_end" length="${eff_length/2}" color="green" />
   <xacro:FIXED_JOINT parent="shaft" child="kinect">
-    <origin xyz="0 0.1 0" />
+    <origin xyz="0 0.265 0" />
   </xacro:FIXED_JOINT>
   <xacro:PLAIN_LINK name="kinect" color="green" />

Commit message: Replace hoge.xacro to arcsys2.xacro

File: src/arcsys2_description/urdf/arcsys2.xacro (robot description, xacro)
@@ -5,68 +5,80 @@
   <material name="green"> <color rgba="${  0/255} ${255/255} ${  0/255} 1.0" /> </material>
   <material name="blue">  <color rgba="${  0/255} ${  0/255} ${255/255} 1.0" /> </material>
-<!-- Property -->
   <xacro:property name="pi" value="3.1415926535897931" />
-  <xacro:property name="default_size" value="0.1" />
-  <xacro:property name="rail_length"  value="3.600" /> <!-- OK? -->
-  <xacro:property name="shaft_height" value="1.350" />
-  <xacro:property name="arm0_length"  value="0.125" />
-  <xacro:property name="arm1_length"  value="0.216" /> <!-- OK? -->
-  <xacro:property name="arm2_length"  value="0.199" /> <!-- OK? -->
-  <xacro:property name="eff_length"   value="0.225" /> <!-- OK? -->
-<!-- LINK and JOINT -->
-  <xacro:PLAIN_LINK name="rail" width="${rail_length*2}" />
-  <xacro:PRISMATIC_JOINT parent="rail" child="shaft" y="1" lower="${-1*rail_length}" upper="${rail_length}">
-    <origin xyz="0 0 ${shaft_height/2}"/>
-    <!-- これのZ座標がキネクトの高度がこれに依存しているので注意 -->
+  <xacro:property name="default_size" value="0.100" />
+  <xacro:property name="arm_init" value="0.200" />
+  <xacro:property name="rail_depth"  value="${default_size}" />
+  <xacro:property name="rail_width"  value="3.600" />
+  <xacro:property name="rail_height" value="${default_size}" />
+  <xacro:property name="base_depth"  value="1.000" />
+  <xacro:property name="base_width"  value="0.850" />
+  <xacro:property name="base_height" value="1.000" />
+  <xacro:property name="shaft_depth"  value="${default_size}" />
+  <xacro:property name="shaft_width"  value="${default_size}" />
+  <xacro:property name="shaft_height" value="1.000" />
+  <xacro:property name="arm0_depth"  value="0.125" />
+  <xacro:property name="arm0_width"  value="${default_size}" />
+  <xacro:property name="arm0_height" value="${default_size}" />
+  <xacro:property name="arm1_depth"  value="0.216" />
+  <xacro:property name="arm1_width"  value="${default_size}" />
+  <xacro:property name="arm1_height" value="${default_size}" />
+  <xacro:property name="arm2_depth"  value="0.199" />
+  <xacro:property name="arm2_width"  value="${default_size}" />
+  <xacro:property name="arm2_height" value="${default_size}" />
+  <xacro:property name="effector_depth"  value="0.225" />
+  <xacro:property name="effector_width"  value="${default_size}" />
+  <xacro:property name="effector_height" value="${default_size}" />
+  <xacro:property name="kinect_offset_x" value="${default_size}" />
+  <xacro:property name="kinect_offset_y" value="0.265" />
+  <xacro:property name="kinect_offset_z" value="${default_size}" />
+  <xacro:property name="kinect_depth"  value="${default_size}" />
+  <xacro:property name="kinect_width"  value="${default_size}" />
+  <xacro:property name="kinect_height" value="${default_size}" />
+  <xacro:PLAIN_LINK name="rail" depth="${rail_depth}" width="${rail_width}" height="${rail_height}" />
+  <xacro:PRISMATIC_JOINT parent="rail" child="base" y="1" lower="${-1*rail_width}" upper="${rail_width}">
+    <origin xyz="0 0 ${base_height/2}" />
   </xacro:PRISMATIC_JOINT>
-  <xacro:PLAIN_LINK name="shaft" height="${shaft_height}" color="red"/>
-  <xacro:PRISMATIC_JOINT parent="shaft" child="arm0" z="1" lower="-0.1" upper="0.1">
-    <origin xyz="${default_size/2} 0 ${shaft_height/4}"/>
-    <!-- ここのdefault_size -> シャフトの奥行き -->
-    <!-- zは初期位置以外の意味は無いと思われる -->
+  <xacro:PLAIN_LINK name="base" depth="${base_depth}" width="${base_width}" height="${base_height}" />
+  <xacro:FIXED_JOINT parent="base" child="kinect">
+    <origin xyz="${kinect_offset_x} ${kinect_offset_y} ${kinect_offset_z}" />
+  </xacro:FIXED_JOINT>
+  <xacro:PLAIN_LINK name="kinect" depth="${kinect_depth}" width="${kinect_width}" height="${kinect_height}" />
+  <xacro:FIXED_JOINT parent="base" child="shaft">
+    <origin xyz="0 0 ${shaft_height/2}" />
+  </xacro:FIXED_JOINT>
+  <xacro:PLAIN_LINK name="shaft" depth="${shaft_depth}" width="${shaft_width}" height="${shaft_height}" />
+  <xacro:PRISMATIC_JOINT parent="shaft" child="arm0" z="1" lower="${-default_size}" upper="${default_size}">
+    <origin xyz="${shaft_depth/2} 0 ${arm_init}" />
   </xacro:PRISMATIC_JOINT>
-  <xacro:SCARA_LINK name="arm0" length="${arm0_length}" color="green"/>
-  <xacro:SCARA_JOINT parent="arm0" child="arm1" parent_length="${arm0_length}"/>
-  <xacro:SCARA_LINK name="arm1" length="${arm1_length}" color="blue"/>
-  <xacro:SCARA_JOINT parent="arm1" child="arm2" parent_length="${arm1_length}"/>
-  <xacro:SCARA_LINK name="arm2" length="${arm2_length}" color="red"/>
-  <xacro:SCARA_JOINT parent="arm2" child="effector_base" parent_length="${arm2_length}"/>
-  <xacro:SCARA_LINK name="effector_base" length="${eff_length/2}" color="green"/>
-  <xacro:WRIST_JOINT parent="effector_base" child="effector_end" parent_length="${eff_length/2}" />
-  <xacro:SCARA_LINK name="effector_end" length="${eff_length/2}" color="green" />
-  <xacro:FIXED_JOINT parent="shaft" child="kinect">
-    <origin xyz="0 0.265 0" />
-  </xacro:FIXED_JOINT>
-  <xacro:PLAIN_LINK name="kinect" color="green" />
-<!-- Macro Definition -->
-  <xacro:macro name="PLAIN_LINK" params="name width:=${default_size} length:=${default_size} height:=${default_size} color:=white">
+  <xacro:SCARA_LINK name="arm0" depth="${arm0_depth}" width="${arm0_width}" height="${arm0_height}" />
+  <xacro:SCARA_JOINT parent="arm0" child="arm1" parent_depth="${arm0_depth}" />
+  <xacro:SCARA_LINK name="arm1" depth="${arm1_depth}" width="${arm1_width}" height="${arm1_height}" />
+  <xacro:SCARA_JOINT parent="arm1" child="arm2" parent_depth="${arm1_depth}" />
+  <xacro:SCARA_LINK name="arm2" depth="${arm2_depth}" width="${arm2_width}" height="${arm2_height}" />
+  <xacro:SCARA_JOINT parent="arm2" child="effector" parent_depth="${arm2_depth}" />
+  <xacro:SCARA_LINK name="effector" depth="${effector_depth/2}" width="${effector_width}" height="${effector_height}" />
+  <xacro:WRIST_JOINT parent="effector" child="blade" parent_depth="${effector_depth/2}" />
+  <xacro:SCARA_LINK name="blade" depth="${effector_depth/2}" width="${effector_width}" height="${effector_height}" />
+  <xacro:macro name="PLAIN_LINK" params="name width:=${default_size} depth:=${default_size} height:=${default_size} color:=white">
     <link name="${name}">
       <origin xyz="0 0 0"/>
       <visual>
-        <geometry>
-          <box size="${length} ${width} ${height}"/>
-        </geometry>
+        <geometry> <box size="${depth} ${width} ${height}"/> </geometry>
         <material name="${color}"/>
       </visual>
       <collision>
-        <geometry>
-          <box size="${length} ${width} ${height}"/>
-        </geometry>
+        <geometry> <box size="${depth} ${width} ${height}"/> </geometry>
       </collision>
     </link>
   </xacro:macro>
-  <xacro:macro name="SCARA_LINK" params="name width:=${default_size} length:=${default_size} height:=${default_size} color:=white">
+  <xacro:macro name="SCARA_LINK" params="name width:=${default_size} depth:=${default_size} height:=${default_size} color:=white">
     <link name="${name}">
       <visual>
-        <origin xyz="${length/2} 0 0"/>
-        <geometry>
-          <box size="${length} ${width} ${height}"/>
-        </geometry>
+        <origin xyz="${depth/2} 0 0"/>
+        <geometry> <box size="${depth} ${width} ${height}"/> </geometry>
         <material name="${color}"/>
       </visual>
       <collision>
-        <geometry>
-          <box size="${length} ${width} ${height}"/>
-        </geometry>
+        <geometry> <box size="${depth} ${width} ${height}"/> </geometry>
       </collision>
     </link>
@@ -88,7 +100,7 @@
     </joint>
   </xacro:macro>
-  <xacro:macro name="SCARA_JOINT" params="parent child parent_length lower:=${-pi/2} upper:=${pi/2}">
+  <xacro:macro name="SCARA_JOINT" params="parent child parent_depth lower:=${-pi/2} upper:=${pi/2}">
     <joint name="${parent}_to_${child}_joint" type="revolute">
-      <origin xyz="${parent_length} 0 0"/>
+      <origin xyz="${parent_depth} 0 0"/>
       <parent link="${parent}"/>
       <child link="${child}"/>
@@ -97,7 +109,7 @@
     </joint>
   </xacro:macro>
-  <xacro:macro name="WRIST_JOINT" params="parent child parent_length lower:=${-pi/2} upper:=${pi/2}">
+  <xacro:macro name="WRIST_JOINT" params="parent child parent_depth lower:=${-pi/2} upper:=${pi/2}">
     <joint name="${parent}_to_${child}_joint" type="revolute">
-      <origin xyz="${parent_length} 0 0"/>
+      <origin xyz="${parent_depth} 0 0"/>
       <parent link="${parent}"/>
       <child link="${child}"/>
