Commit message: Fix bug

File: src/arcsys2_description/urdf/arcsys2.xacro (robot description, xacro)
@@ -11,10 +11,10 @@
   <xacro:property name="rail_width"  value="3.600" />
   <xacro:property name="rail_height" value="${default_size}" />
-  <xacro:property name="base_depth"  value="1.000" />
+  <xacro:property name="base_depth"  value="0.600" />
   <xacro:property name="base_width"  value="0.850" />
-  <xacro:property name="base_height" value="1.000" />
+  <xacro:property name="base_height" value="0.500" />
   <xacro:property name="shaft_depth"  value="${default_size}" />
   <xacro:property name="shaft_width"  value="${default_size}" />
-  <xacro:property name="shaft_height" value="1.000" />
+  <xacro:property name="shaft_height" value="0.800" />
   <xacro:property name="arm0_depth"  value="0.125" />
   <xacro:property name="arm0_width"  value="${default_size}" />
@@ -35,29 +35,29 @@
   <xacro:property name="kinect_width"  value="${default_size}" />
   <xacro:property name="kinect_height" value="${default_size}" />
-  <xacro:PLAIN_LINK name="rail" depth="${rail_depth}" width="${rail_width}" height="${rail_height}" />
+  <xacro:PLAIN_LINK name="rail" depth="${rail_depth}" width="${rail_width}" height="${rail_height}" color="white" />
   <xacro:PRISMATIC_JOINT parent="rail" child="base" y="1" lower="${-1*rail_width}" upper="${rail_width}">
     <origin xyz="0 0 ${base_height/2}" />
   </xacro:PRISMATIC_JOINT>
-  <xacro:PLAIN_LINK name="base" depth="${base_depth}" width="${base_width}" height="${base_height}" />
+  <xacro:PLAIN_LINK name="base" depth="${base_depth}" width="${base_width}" height="${base_height}" color="red" />
   <xacro:FIXED_JOINT parent="base" child="kinect">
     <origin xyz="${kinect_offset_x} ${kinect_offset_y} ${kinect_offset_z}" />
   </xacro:FIXED_JOINT>
-  <xacro:PLAIN_LINK name="kinect" depth="${kinect_depth}" width="${kinect_width}" height="${kinect_height}" />
+  <xacro:PLAIN_LINK name="kinect" depth="${kinect_depth}" width="${kinect_width}" height="${base_height+kinect_height}" color="green" />
   <xacro:FIXED_JOINT parent="base" child="shaft">
-    <origin xyz="0 0 ${shaft_height/2}" />
+    <origin xyz="-0.15 0 ${shaft_height/2}" />
   </xacro:FIXED_JOINT>
-  <xacro:PLAIN_LINK name="shaft" depth="${shaft_depth}" width="${shaft_width}" height="${shaft_height}" />
+  <xacro:PLAIN_LINK name="shaft" depth="${shaft_depth}" width="${shaft_width}" height="${shaft_height}" color="blue" />
   <xacro:PRISMATIC_JOINT parent="shaft" child="arm0" z="1" lower="${-default_size}" upper="${default_size}">
     <origin xyz="${shaft_depth/2} 0 ${arm_init}" />
   </xacro:PRISMATIC_JOINT>
-  <xacro:SCARA_LINK name="arm0" depth="${arm0_depth}" width="${arm0_width}" height="${arm0_height}" />
+  <xacro:SCARA_LINK name="arm0" depth="${arm0_depth}" width="${arm0_width}" height="${arm0_height}" color="red" />
   <xacro:SCARA_JOINT parent="arm0" child="arm1" parent_depth="${arm0_depth}" />
-  <xacro:SCARA_LINK name="arm1" depth="${arm1_depth}" width="${arm1_width}" height="${arm1_height}" />
+  <xacro:SCARA_LINK name="arm1" depth="${arm1_depth}" width="${arm1_width}" height="${arm1_height}" color="green" />
   <xacro:SCARA_JOINT parent="arm1" child="arm2" parent_depth="${arm1_depth}" />
-  <xacro:SCARA_LINK name="arm2" depth="${arm2_depth}" width="${arm2_width}" height="${arm2_height}" />
+  <xacro:SCARA_LINK name="arm2" depth="${arm2_depth}" width="${arm2_width}" height="${arm2_height}" color="blue" />
   <xacro:SCARA_JOINT parent="arm2" child="effector" parent_depth="${arm2_depth}" />
-  <xacro:SCARA_LINK name="effector" depth="${effector_depth/2}" width="${effector_width}" height="${effector_height}" />
+  <xacro:SCARA_LINK name="effector" depth="${effector_depth/2}" width="${effector_width}" height="${effector_height}" color="red" />
   <xacro:WRIST_JOINT parent="effector" child="blade" parent_depth="${effector_depth/2}" />
-  <xacro:SCARA_LINK name="blade" depth="${effector_depth/2}" width="${effector_width}" height="${effector_height}" />
+  <xacro:SCARA_LINK name="blade" depth="${effector_depth/2}" width="${effector_width}" height="${effector_height}" color="red" />
   <xacro:macro name="PLAIN_LINK" params="name width:=${default_size} depth:=${default_size} height:=${default_size} color:=white">
     <link name="${name}">

Commit message: Regenerate robot description

File: src/arcsys2_description/urdf/arcsys2.xacro (robot description, xacro)
@@ -35,6 +35,6 @@
   <xacro:property name="kinect_width"  value="${default_size}" />
   <xacro:property name="kinect_height" value="${default_size}" />
-  <xacro:PLAIN_LINK name="rail" depth="${rail_depth}" width="${rail_width}" height="${rail_height}" color="white" />
-  <xacro:PRISMATIC_JOINT parent="rail" child="base" y="1" lower="${-1*rail_width}" upper="${rail_width}">
+  <xacro:PLAIN_LINK name="rail" depth="${rail_depth}" width="${rail_width - base_width}" height="${rail_height}" color="white" />
+  <xacro:PRISMATIC_JOINT parent="rail" child="base" y="1" lower="0" upper="${rail_width - base_width}">
     <origin xyz="0 0 ${base_height/2}" />
   </xacro:PRISMATIC_JOINT>
@@ -67,7 +67,7 @@
         <material name="${color}"/>
       </visual>
-      <collision>
-        <geometry> <box size="${depth} ${width} ${height}"/> </geometry>
-      </collision>
+      <!-- <collision>                                                        -->
+      <!--   <geometry> <box size="${depth} ${width} ${height}"/> </geometry> -->
+      <!-- </collision>                                                       -->
     </link>
   </xacro:macro>
@@ -79,7 +79,7 @@
         <material name="${color}"/>
       </visual>
-      <collision>
-        <geometry> <box size="${depth} ${width} ${height}"/> </geometry>
-      </collision>
+      <!-- <collision>                                                        -->
+      <!--   <geometry> <box size="${depth} ${width} ${height}"/> </geometry> -->
+      <!-- </collision>                                                       -->
     </link>
   </xacro:macro>

Commit message: Cleanup

File: src/arcsys2_description/urdf/arcsys2.xacro (robot description, xacro)
@@ -1,8 +1,10 @@
 <?xml version="1.0"?>
 <robot xmlns:xacro="http://ros.org/wiki/xacro" name="arcsys2">
+<!-- MATERIAL -->
   <material name="white"> <color rgba="${255/255} ${255/255} ${255/255} 1.0" /> </material>
   <material name="red">   <color rgba="${255/255} ${  0/255} ${  0/255} 1.0" /> </material>
   <material name="green"> <color rgba="${  0/255} ${255/255} ${  0/255} 1.0" /> </material>
   <material name="blue">  <color rgba="${  0/255} ${  0/255} ${255/255} 1.0" /> </material>
+<!-- PROPERTY -->
   <xacro:property name="pi" value="3.1415926535897931" />
   <xacro:property name="default_size" value="0.100" />
@@ -35,17 +37,26 @@
   <xacro:property name="kinect_width"  value="${default_size}" />
   <xacro:property name="kinect_height" value="${default_size}" />
-  <xacro:PLAIN_LINK name="rail" depth="${rail_depth}" width="${rail_width - base_width}" height="${rail_height}" color="white" />
+<!-- LINK AND JOINT -->
+  <xacro:PLAIN_LINK name="rail" depth="${rail_depth}" width="${rail_width-base_width}" height="${rail_height}">
+    <origin xyz="${rail_width-base_width} 0 0" />
+  </xacro:PLAIN_LINK>
   <xacro:PRISMATIC_JOINT parent="rail" child="base" y="1" lower="0" upper="${rail_width - base_width}">
     <origin xyz="0 0 ${base_height/2}" />
   </xacro:PRISMATIC_JOINT>
-  <xacro:PLAIN_LINK name="base" depth="${base_depth}" width="${base_width}" height="${base_height}" color="red" />
+  <xacro:PLAIN_LINK name="base" depth="${base_depth}" width="${base_width}" height="${base_height}" color="red">
+    <origin xyz="0 0 0" />
+  </xacro:PLAIN_LINK>
   <xacro:FIXED_JOINT parent="base" child="kinect">
     <origin xyz="${kinect_offset_x} ${kinect_offset_y} ${kinect_offset_z}" />
   </xacro:FIXED_JOINT>
-  <xacro:PLAIN_LINK name="kinect" depth="${kinect_depth}" width="${kinect_width}" height="${base_height+kinect_height}" color="green" />
+  <xacro:PLAIN_LINK name="kinect" depth="${kinect_depth}" width="${kinect_width}" height="${kinect_height}" color="green">
+    <origin xyz="0 0 ${base_height}" />
+  </xacro:PLAIN_LINK>
   <xacro:FIXED_JOINT parent="base" child="shaft">
     <origin xyz="-0.15 0 ${shaft_height/2}" />
   </xacro:FIXED_JOINT>
-  <xacro:PLAIN_LINK name="shaft" depth="${shaft_depth}" width="${shaft_width}" height="${shaft_height}" color="blue" />
+  <xacro:PLAIN_LINK name="shaft" depth="${shaft_depth}" width="${shaft_width}" height="${shaft_height}" color="blue">
+    <origin xyz="0 0 0" />
+  </xacro:PLAIN_LINK>
   <xacro:PRISMATIC_JOINT parent="shaft" child="arm0" z="1" lower="${-default_size}" upper="${default_size}">
     <origin xyz="${shaft_depth/2} 0 ${arm_init}" />
@@ -60,26 +71,21 @@
   <xacro:WRIST_JOINT parent="effector" child="blade" parent_depth="${effector_depth/2}" />
   <xacro:SCARA_LINK name="blade" depth="${effector_depth/2}" width="${effector_width}" height="${effector_height}" color="red" />
-  <xacro:macro name="PLAIN_LINK" params="name width:=${default_size} depth:=${default_size} height:=${default_size} color:=white">
+<!-- MACRO DEFINITION -->
+  <xacro:macro name="PLAIN_LINK" params="name width:=${default_size} depth:=${default_size} height:=${default_size} color:=white *origin">
     <link name="${name}">
-      <origin xyz="0 0 0"/>
+      <xacro:insert_block name="origin" />
       <visual>
-        <geometry> <box size="${depth} ${width} ${height}"/> </geometry>
-        <material name="${color}"/>
+        <geometry> <box size="${depth} ${width} ${height}" /> </geometry>
+        <material name="${color}" />
       </visual>
-      <!-- <collision>                                                        -->
-      <!--   <geometry> <box size="${depth} ${width} ${height}"/> </geometry> -->
-      <!-- </collision>                                                       -->
     </link>
   </xacro:macro>
-  <xacro:macro name="SCARA_LINK" params="name width:=${default_size} depth:=${default_size} height:=${default_size} color:=white">
+  <xacro:macro name="SCARA_LINK" params="name width:=${default_size} depth:=${default_size} height:=${default_size} offset_y:=0 offset_z:=0 color:=white">
     <link name="${name}">
       <visual>
-        <origin xyz="${depth/2} 0 0"/>
-        <geometry> <box size="${depth} ${width} ${height}"/> </geometry>
-        <material name="${color}"/>
+        <origin xyz="${depth/2} ${offset_y} ${offset_z}" />
+        <geometry> <box size="${depth} ${width} ${height}" /> </geometry>
+        <material name="${color}" />
       </visual>
-      <!-- <collision>                                                        -->
-      <!--   <geometry> <box size="${depth} ${width} ${height}"/> </geometry> -->
-      <!-- </collision>                                                       -->
     </link>
   </xacro:macro>

Commit message: Add new xacro macro "REVOLUTE_JOINT"

File: src/arcsys2_description/urdf/arcsys2.xacro (robot description, xacro)
@@ -8,6 +8,10 @@
 <!-- PROPERTY -->
   <xacro:property name="pi" value="3.1415926535897931" />
-  <xacro:property name="default_size" value="0.100" />
-  <xacro:property name="arm_init" value="0.200" />
+  <xacro:property name="default_size"     value="0.100" />
+  <xacro:property name="default_lower"    value="${-pi/2}" />
+  <xacro:property name="default_upper"    value="${+pi/2}" />
+  <xacro:property name="default_effort"   value="1.0" />
+  <xacro:property name="default_velocity" value="1.0" />
+  <xacro:property name="arm_init"     value="0.200" />
   <xacro:property name="rail_depth"  value="${default_size}" />
   <xacro:property name="rail_width"  value="3.600" />
@@ -31,15 +35,16 @@
   <xacro:property name="effector_width"  value="${default_size}" />
   <xacro:property name="effector_height" value="${default_size}" />
-  <xacro:property name="kinect_offset_x" value="${default_size}" />
-  <xacro:property name="kinect_offset_y" value="0.265" />
-  <xacro:property name="kinect_offset_z" value="${default_size}" />
+  <xacro:property name="kinect_offx" value="${default_size}" />
+  <xacro:property name="kinect_offy" value="0.265" />
+  <xacro:property name="kinect_offz" value="${default_size}" />
   <xacro:property name="kinect_depth"  value="${default_size}" />
   <xacro:property name="kinect_width"  value="${default_size}" />
   <xacro:property name="kinect_height" value="${default_size}" />
 <!-- LINK AND JOINT -->
-  <xacro:PLAIN_LINK name="rail" depth="${rail_depth}" width="${rail_width-base_width}" height="${rail_height}">
-    <origin xyz="${rail_width-base_width} 0 0" />
+  <xacro:PLAIN_LINK name="rail" depth="${rail_depth}" width="${rail_width*2}" height="${rail_height}">
+    <origin xyz="${rail_width} 0 0" />
   </xacro:PLAIN_LINK>
-  <xacro:PRISMATIC_JOINT parent="rail" child="base" y="1" lower="0" upper="${rail_width - base_width}">
+  <xacro:PRISMATIC_JOINT parent="rail" child="base" y="1" lower="0" upper="${rail_width-base_width/2}">
+  <!-- <xacro:PRISMATIC_JOINT parent="rail" child="base" y="1" lower="${rail_width-base_width/2}" upper="0"> -->
     <origin xyz="0 0 ${base_height/2}" />
   </xacro:PRISMATIC_JOINT>
@@ -48,8 +53,8 @@
   </xacro:PLAIN_LINK>
   <xacro:FIXED_JOINT parent="base" child="kinect">
-    <origin xyz="${kinect_offset_x} ${kinect_offset_y} ${kinect_offset_z}" />
+    <origin xyz="${kinect_offx} ${kinect_offy} ${kinect_offz}" />
   </xacro:FIXED_JOINT>
   <xacro:PLAIN_LINK name="kinect" depth="${kinect_depth}" width="${kinect_width}" height="${kinect_height}" color="green">
-    <origin xyz="0 0 ${base_height}" />
+    <origin xyz="0 0 ${rail_height+base_height}" />
   </xacro:PLAIN_LINK>
   <xacro:FIXED_JOINT parent="base" child="shaft">
@@ -69,5 +74,8 @@
   <xacro:SCARA_JOINT parent="arm2" child="effector" parent_depth="${arm2_depth}" />
   <xacro:SCARA_LINK name="effector" depth="${effector_depth/2}" width="${effector_width}" height="${effector_height}" color="red" />
-  <xacro:WRIST_JOINT parent="effector" child="blade" parent_depth="${effector_depth/2}" />
+  <!-- <xacro:WRIST_JOINT parent="effector" child="blade" parent_depth="${effector_depth/2}" lower="0" upper="pi*3/4" /> -->
+  <xacro:REVOLUTE_JOINT parent="effector" child="blade" axisx="1" lower="0" upper="${pi*3/4}">
+    <origin xyz="${effector_depth/2} 0 0" />
+  </xacro:REVOLUTE_JOINT>
   <xacro:SCARA_LINK name="blade" depth="${effector_depth/2}" width="${effector_width}" height="${effector_height}" color="red" />
 <!-- MACRO DEFINITION -->
@@ -81,8 +89,8 @@
     </link>
   </xacro:macro>
-  <xacro:macro name="SCARA_LINK" params="name width:=${default_size} depth:=${default_size} height:=${default_size} offset_y:=0 offset_z:=0 color:=white">
+  <xacro:macro name="SCARA_LINK" params="name width:=${default_size} depth:=${default_size} height:=${default_size} offy:=0 offz:=0 color:=white">
     <link name="${name}">
       <visual>
-        <origin xyz="${depth/2} ${offset_y} ${offset_z}" />
+        <origin xyz="${depth/2} ${offy} ${offz}" />
         <geometry> <box size="${depth} ${width} ${height}" /> </geometry>
         <material name="${color}" />
@@ -92,7 +100,7 @@
   <xacro:macro name="FIXED_JOINT" params="parent child *origin">
     <joint name="${parent}_to_${child}_joint" type="fixed">
-      <xacro:insert_block name="origin"/>
-      <parent link="${parent}"/>
-      <child link="${child}"/>
+      <xacro:insert_block name="origin" />
+      <parent link="${parent}" />
+      <child link="${child}" />
     </joint>
   </xacro:macro>
@@ -124,3 +132,12 @@
     </joint>
   </xacro:macro>
+  <xacro:macro name="REVOLUTE_JOINT" params="parent child *origin axisx:=0 axisy:=0 axisz:=0 lower:=${default_lower} upper:=${default_upper} effort:=${default_effort} velocity:=${default_velocity}">
+    <joint name="${parent}_to_${child}_joint" type="revolute">
+      <xacro:insert_block name="origin" />
+      <parent link="${parent}" />
+      <child link="${child}" />
+      <axis xyz="${axisx} ${axisy} ${axisz}" />
+      <limit lower="${lower}" upper="${upper}" effort="${effort}" velocity="${velocity}" />
+    </joint>
+  </xacro:macro>
 </robot>

Commit message: Chage SCARA_JOINT and WRIST_JOINT to REVOLUTE_JOINT

File: src/arcsys2_description/urdf/arcsys2.xacro (robot description, xacro)
@@ -68,11 +68,16 @@
   </xacro:PRISMATIC_JOINT>
   <xacro:SCARA_LINK name="arm0" depth="${arm0_depth}" width="${arm0_width}" height="${arm0_height}" color="red" />
-  <xacro:SCARA_JOINT parent="arm0" child="arm1" parent_depth="${arm0_depth}" />
+  <xacro:REVOLUTE_JOINT parent="arm0" child="arm1" axisz="1">
+    <origin xyz="${arm0_depth} 0 0" />
+  </xacro:REVOLUTE_JOINT>
   <xacro:SCARA_LINK name="arm1" depth="${arm1_depth}" width="${arm1_width}" height="${arm1_height}" color="green" />
-  <xacro:SCARA_JOINT parent="arm1" child="arm2" parent_depth="${arm1_depth}" />
+  <xacro:REVOLUTE_JOINT parent="arm1" child="arm2" axisz="1">
+    <origin xyz="${arm1_depth} 0 0" />
+  </xacro:REVOLUTE_JOINT>
   <xacro:SCARA_LINK name="arm2" depth="${arm2_depth}" width="${arm2_width}" height="${arm2_height}" color="blue" />
-  <xacro:SCARA_JOINT parent="arm2" child="effector" parent_depth="${arm2_depth}" />
+  <xacro:REVOLUTE_JOINT parent="arm2" child="effector" axisz="1">
+    <origin xyz="${arm2_depth} 0 0" />
+  </xacro:REVOLUTE_JOINT>
   <xacro:SCARA_LINK name="effector" depth="${effector_depth/2}" width="${effector_width}" height="${effector_height}" color="red" />
-  <!-- <xacro:WRIST_JOINT parent="effector" child="blade" parent_depth="${effector_depth/2}" lower="0" upper="pi*3/4" /> -->
   <xacro:REVOLUTE_JOINT parent="effector" child="blade" axisx="1" lower="0" upper="${pi*3/4}">
     <origin xyz="${effector_depth/2} 0 0" />
@@ -114,22 +119,4 @@
     </joint>
   </xacro:macro>
-  <xacro:macro name="SCARA_JOINT" params="parent child parent_depth lower:=${-pi/2} upper:=${pi/2}">
-    <joint name="${parent}_to_${child}_joint" type="revolute">
-      <origin xyz="${parent_depth} 0 0"/>
-      <parent link="${parent}"/>
-      <child link="${child}"/>
-      <axis xyz="0 0 1"/>
-      <limit lower="${lower}" upper="${upper}" effort="1" velocity="1"/>
-    </joint>
-  </xacro:macro>
-  <xacro:macro name="WRIST_JOINT" params="parent child parent_depth lower:=${-pi/2} upper:=${pi/2}">
-    <joint name="${parent}_to_${child}_joint" type="revolute">
-      <origin xyz="${parent_depth} 0 0"/>
-      <parent link="${parent}"/>
-      <child link="${child}"/>
-      <axis xyz="1 0 0"/>
-      <limit lower="${lower}" upper="${upper}" effort="1" velocity="1"/>
-    </joint>
-  </xacro:macro>
   <xacro:macro name="REVOLUTE_JOINT" params="parent child *origin axisx:=0 axisy:=0 axisz:=0 lower:=${default_lower} upper:=${default_upper} effort:=${default_effort} velocity:=${default_velocity}">
     <joint name="${parent}_to_${child}_joint" type="revolute">

Commit message: Update kinect link configs

File: src/arcsys2_description/urdf/arcsys2.xacro (robot description, xacro)
@@ -20,4 +20,7 @@
   <xacro:property name="base_width"  value="0.850" />
   <xacro:property name="base_height" value="0.500" />
+  <xacro:property name="shaft_offx"   value="-0.15" />
+  <xacro:property name="shaft_offy"   value="0" />
+  <xacro:property name="shaft_offz"   value="0" />
   <xacro:property name="shaft_depth"  value="${default_size}" />
   <xacro:property name="shaft_width"  value="${default_size}" />
@@ -35,7 +38,7 @@
   <xacro:property name="effector_width"  value="${default_size}" />
   <xacro:property name="effector_height" value="${default_size}" />
-  <xacro:property name="kinect_offx" value="${default_size}" />
+  <xacro:property name="kinect_offx" value="0" />
   <xacro:property name="kinect_offy" value="0.265" />
-  <xacro:property name="kinect_offz" value="${default_size}" />
+  <xacro:property name="kinect_offz" value="0" />
   <xacro:property name="kinect_depth"  value="${default_size}" />
   <xacro:property name="kinect_width"  value="${default_size}" />
@@ -53,11 +56,11 @@
   </xacro:PLAIN_LINK>
   <xacro:FIXED_JOINT parent="base" child="kinect">
-    <origin xyz="${kinect_offx} ${kinect_offy} ${kinect_offz}" />
+    <origin xyz="${kinect_offx} ${kinect_offy} ${kinect_offz+base_height/2}" />
   </xacro:FIXED_JOINT>
   <xacro:PLAIN_LINK name="kinect" depth="${kinect_depth}" width="${kinect_width}" height="${kinect_height}" color="green">
-    <origin xyz="0 0 ${rail_height+base_height}" />
+    <origin xyz="0 0 0" />
   </xacro:PLAIN_LINK>
   <xacro:FIXED_JOINT parent="base" child="shaft">
-    <origin xyz="-0.15 0 ${shaft_height/2}" />
+    <origin xyz="${shaft_offx} ${shaft_offy} ${shaft_offz+shaft_height/2}" />
   </xacro:FIXED_JOINT>
   <xacro:PLAIN_LINK name="shaft" depth="${shaft_depth}" width="${shaft_width}" height="${shaft_height}" color="blue">
@@ -85,5 +88,5 @@
   <xacro:SCARA_LINK name="blade" depth="${effector_depth/2}" width="${effector_width}" height="${effector_height}" color="red" />
 <!-- MACRO DEFINITION -->
-  <xacro:macro name="PLAIN_LINK" params="name width:=${default_size} depth:=${default_size} height:=${default_size} color:=white *origin">
+  <xacro:macro name="PLAIN_LINK" params="name *origin width:=${default_size} depth:=${default_size} height:=${default_size} color:=white">
     <link name="${name}">
       <xacro:insert_block name="origin" />
