Commit message: Update some properties to actual size

File: src/arcsys2_description/urdf/arcsys2.xacro (robot description, xacro)
@@ -11,19 +11,19 @@
   <xacro:property name="default_lower"    value="${-pi/2}" />
   <xacro:property name="default_upper"    value="${+pi/2}" />
-  <xacro:property name="default_effort"   value="1.0" />
-  <xacro:property name="default_velocity" value="1.0" />
-  <xacro:property name="arm_init"     value="0.200" />
+  <xacro:property name="default_effort"   value="1.000" />
+  <xacro:property name="default_velocity" value="1.000" />
+  <xacro:property name="arm_init"     value="0" />
   <xacro:property name="rail_depth"  value="${default_size}" />
   <xacro:property name="rail_width"  value="3.600" />
-  <xacro:property name="rail_height" value="${default_size}" />
-  <xacro:property name="base_depth"  value="0.600" />
-  <xacro:property name="base_width"  value="0.850" />
-  <xacro:property name="base_height" value="0.500" />
-  <xacro:property name="shaft_offx"   value="-0.15" />
+  <xacro:property name="rail_height" value="0.060" />
+  <xacro:property name="base_depth"  value="0.580" />
+  <xacro:property name="base_width"  value="0.750" />
+  <xacro:property name="base_height" value="0.520" />
+  <xacro:property name="shaft_offx"   value="-0.120" />
   <xacro:property name="shaft_offy"   value="0" />
   <xacro:property name="shaft_offz"   value="0" />
   <xacro:property name="shaft_depth"  value="${default_size}" />
   <xacro:property name="shaft_width"  value="${default_size}" />
-  <xacro:property name="shaft_height" value="0.800" />
+  <xacro:property name="shaft_height" value="0.850" />
   <xacro:property name="arm0_depth"  value="0.125" />
   <xacro:property name="arm0_width"  value="${default_size}" />
@@ -38,7 +38,7 @@
   <xacro:property name="effector_width"  value="${default_size}" />
   <xacro:property name="effector_height" value="${default_size}" />
-  <xacro:property name="kinect_offx" value="0" />
-  <xacro:property name="kinect_offy" value="0.265" />
-  <xacro:property name="kinect_offz" value="0" />
+  <xacro:property name="kinect_offx" value="-0.250" />
+  <xacro:property name="kinect_offy" value="0.300" />
+  <xacro:property name="kinect_offz" value="0.360" />
   <xacro:property name="kinect_depth"  value="${default_size}" />
   <xacro:property name="kinect_width"  value="${default_size}" />
@@ -67,5 +67,5 @@
     <origin xyz="0 0 0" />
   </xacro:PLAIN_LINK>
-  <xacro:PRISMATIC_JOINT parent="shaft" child="arm0" z="1" lower="${-default_size}" upper="${default_size}">
+  <xacro:PRISMATIC_JOINT parent="shaft" child="arm0" z="1" lower="0" upper="0.30">
     <origin xyz="${shaft_depth/2} 0 ${arm_init}" />
   </xacro:PRISMATIC_JOINT>
